File: EVALTOLTDC48V3KWTOBO2_SinglePhase/Current amplifier.kicad_sch (KiCad schematic)
At the start: 11 parts

Commit message: Change 4
Other:
- moved on the sheet: OP1
Changed lines of the file:
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@@
 	(symbol
 		(lib_id "AD8615AUJZ:AD8615AUJZ")
-		(at 133.35 80.645 0)
+		(at 190.5 52.07 0)
 		(unit 1)
 		(exclude_from_sim no)
@@
 		(dnp no)
 		(property "Reference" "OP1"
-			(at 136.0932 94.9198 0)
+			(at 193.2432 66.3448 0)
 			(effects
 				(font
@@
 		)
 		(property "Value" "AD8615AUJZ"
-			(at 140.208 101.9302 0)
+			(at 197.358 73.3552 0)
 			(effects
 				(font
@@
 		)
 		(property "Footprint" "AD8615AUJZ:SOT95P280X100-5N"
-			(at 133.35 80.645 0)
+			(at 190.5 52.07 0)
 			(effects
 				(font
@@
 		)
 		(property "Datasheet" ""
-			(at 133.35 80.645 0)
+			(at 190.5 52.07 0)
 			(effects
 				(font
@@
 		)
 		(property "Description" "\nPrecision 20 MHz CMOS Single RRIO Operational Amplifier\n"
-			(at 133.35 80.645 0)
+			(at 190.5 52.07 0)
 			(effects
 				(font
@@
 		)
 		(property "MF" "Analog Devices"
-			(at 133.35 80.645 0)
+			(at 190.5 52.07 0)
 			(effects
 				(font
@@
 		)
 		(property "PACKAGE" "SOT-23-5"
-			(at 133.35 80.645 0)
+			(at 190.5 52.07 0)
 			(effects
 				(font
@@
 		)
 		(property "MPN" "AD8615AUJZ"
-			(at 133.35 80.645 0)
+			(at 190.5 52.07 0)
 			(effects
 				(font
@@
 		)
 		(property "Price" "None"
-			(at 133.35 80.645 0)
+			(at 190.5 52.07 0)
 			(effects
 				(font
@@
 		)
 		(property "Package" "TSOT-5 Analog Devices"
-			(at 133.35 80.645 0)
+			(at 190.5 52.07 0)
 			(effects
 				(font
@@
 		)
 		(property "OC_FARNELL" "9079408"
-			(at 133.35 80.645 0)
+			(at 190.5 52.07 0)
 			(effects
 				(font
@@
 		)
 		(property "SnapEDA_Link" "https://www.snapeda.com/parts/AD8615AUJZ-REEL7/Analog+Devices/view-part/?ref=snap"
-			(at 133.35 80.645 0)
+			(at 190.5 52.07 0)
 			(effects
 				(font
@@
 		)
 		(property "MP" "AD8615AUJZ-REEL7"
-			(at 133.35 80.645 0)
+			(at 190.5 52.07 0)
 			(effects
 				(font
@@
 		)
 		(property "Purchase-URL" "https://www.snapeda.com/api/url_track_click_mouser/?unipart_id=45535&manufacturer=Analog Devices&part_name=AD8615AUJZ-REEL7&search_term=ad8615"
-			(at 133.35 80.645 0)
+			(at 190.5 52.07 0)
 			(effects
 				(font
@@
 		)
 		(property "SUPPLIER" "Analog Devices"
-			(at 133.35 80.645 0)
+			(at 190.5 52.07 0)
 			(effects
 				(font
@@
 		)
 		(property "OC_NEWARK" "31M4569"
-			(at 133.35 80.645 0)
+			(at 190.5 52.07 0)
 			(effects
 				(font
@@
 		)
 		(property "Availability" "In Stock"
-			(at 133.35 80.645 0)
+			(at 190.5 52.07 0)
 			(effects
 				(font
@@
 		)
 		(property "Check_prices" "https://www.snapeda.com/parts/AD8615AUJZ-REEL7/Analog+Devices/view-part/?ref=eda"
-			(at 133.35 80.645 0)
+			(at 190.5 52.07 0)
 			(effects
 				(font
@@
 		)
 		(property "Description_1" "\nPrecision 20 MHz CMOS Single RRIO Operational Amplifier\n"
-			(at 133.35 80.645 0)
+			(at 190.5 52.07 0)
 			(effects
 				(font
@@
 		(on_board yes)
 		(dnp no)
-		(fields_autoplaced yes)
 		(property "Reference" "R45"
-			(at 142.24 74.93 0)
-			(effects
-				(font
+			(at 136.652 65.786 0)
+			(effects
+				(font
