File: EVALTOLTDC48V3KWTOBO2_SinglePhase/Power Board Connector.kicad_sch (KiCad schematic)
At the start: 18 parts, among them J12 Direction Switch, Q7 IRLML6346, U12 PCN10C-32S-2.54DS(72)

Commit message: Change 4
Connections:
- net GNDS: now also C81.1, C82.2
- net at R76.1, U12. (B9): now also C81.2
- net at R75.1, RT1.1 (V_{DD}): now also C82.1
- no-connect marks 12 -> 20
Other:
- moved on the sheet: C81, C82, U12
