File: EVALTOLTDC48V3KWTOBO2_SinglePhase/Current Comparator & Latch.kicad_sch (KiCad schematic)
At the start: 29 parts, among them Q8 IRLML6346, U11 LMV331, U13 SN74LVC2G74DCUR

Commit message: Change 6
Parts:
- added D13, D14: 500mA/30V/TSLP-2-17, just-footprints:PMEG3005ELD315, symbol PMEG3005ELD_315:PMEG3005ELD,315
- added R65, R66: 0 0402, symbol Device:R
- C74, C93: footprint just-footprints:CAPC17595_95N_KEM -> All Footprints:C74,C93 (1); symbol C0603C105K3RAC7411:C0603C105K3RAC7411 -> Device:C
- C75: footprint just-footprints:CAPC17795_95N_KEM -> All Footprints:C75,C78,C92 (3); symbol C0603X104M3RAUTO:C0603X104M3RACTU -> Device:C
- C76: footprint (none) -> All Footprints:C76 (1)
- C77: footprint just-footprints:CAPC10555_55N_KEM -> All Footprints:C77,C79 (1); symbol C0603C101K3RACAUTO:C0402C101K3RACTU -> Device:C
- C78, C92: footprint (none) -> All Footprints:C75,C78,C92 (3)
- Ct1: renamed from C79; footprint just-footprints:CAPC10555_55N_KEM -> All Footprints:C77,C79 (1); symbol C0603C101K3RACAUTO:C0402C101K3RACTU -> Device:C
- LED4: footprint (none) -> All Footprints:LED4
- POT2: footprint just-footprints:SM42TW503 -> All Footprints:POT2; symbol SM-42TW503:SM-42TW503 -> Device:R_Potentiometer; Height 5.6 -> (none); Manufacturer_Name Nidec Copal -> (none); Manufacturer_Part_Number SM-42TW503 -> (none); Mouser Part Number 229-SM-42TW503 -> (none); Mouser Price/Stock https://www.mouser.co.uk/ProductDetail/Nidec-Components/SM-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 -> (none)
- R63: symbol PFR05S-103-FNH:PFR05S-103-FNH -> 2024-05-10_08-55-23:PFR05S-103-FNH
- R64: footprint just-footprints:RC0402N_PAN -> (none); symbol ERJ-2GE0R00X:ERJ-2GE0R00X -> Device:R
- R67, R68, R71: footprint just-footprints:RES_RCA0603_VIS -> All Footprints:RES_RCA0603_VIS; symbol RCA06031K00FKEAHP:RCA06031K00FKEAHP -> Device:R
- R69: footprint ERJP03_PA3_(0603) -> All Footprints:ERJP03_PA3__0603_; symbol ERJ-PA3J100V:ERJ-PA3J100V -> Device:R; Height 0.55 -> (none); Manufacturer_Name Panasonic -> (none); Manufacturer_Part_Number ERJ-PA3J100V -> (none); Mouser Part Number 667-ERJ-PA3J100V -> (none); Mouser Price/Stock https://www.mouser.co.uk/ProductDetail/Panasonic/ERJ-PA3J10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 -> (none)
- R70: footprint (none) -> All Footprints:R70 (1)
- R87, R88: footprint (none) -> All Footprints:RES_ERJUP3_PAN
- R89, R90: footprint (none) -> All Footprints:RESC1508X50N
Connections:
- net +5V: now also R67.1, R69.1, R71.1; no longer R67.2, R69.2
- net GND: now also C77.2, C93.2, Ct1.2
- net at OP5.1 (OUT), OP5.4 (-IN), TP4.1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: now also C77.1
- net at C74.1, OP5.3 (+IN), POT2.1: now also R67.2; no longer R67.1
- net at C75.1, OP5.5 (V+): now also R69.2; no longer R69.1
- net at R70.2, TP5.1, U11.4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: now also Ct1.1, R71.2
- net at R89.2, U13.6 (~{CLR}): now also C93.1
- net at C76.1, D12.1 (K), R63.2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: now also D13.1 (K), D14.1 (K)
- new net: D14.2 (A), R66.2
- new net: D13.2 (A), R65.2
- new net I_PHASE_V: R65.1
- new net I_PHASE_W: R66.1
Other:
- moved on the sheet: D12, R63
