File: EVALTOLTDC48V3KWTOBO2_SinglePhase/Current Comparator & Latch_NOTALP.kicad_sch (KiCad schematic)
At the start: 33 parts, among them Q8 IRLML6346, U11 LMV331, U13 SN74LVC2G74DCUR

Commit message: Change 6
Parts:
- removed D13, D14: 500mA/30V/TSLP-2-17, PMEG3005ELD315, symbol PMEG3005ELD_315:PMEG3005ELD,315
- removed R65, R66: 0 0402, symbol Device:R
- C74, C93: footprint All Footprints:C74,C93 (1) -> just-footprints:CAPC17595_95N_KEM; symbol Device:C -> C0603C105K3RAC7411:C0603C105K3RAC7411
- C75: footprint All Footprints:C75,C78,C92 (3) -> just-footprints:CAPC17795_95N_KEM; symbol Device:C -> C0603X104M3RAUTO:C0603X104M3RACTU
- C76: footprint All Footprints:C76 (1) -> (none)
- C77: footprint All Footprints:C77,C79 (1) -> just-footprints:CAPC10555_55N_KEM; symbol Device:C -> C0603C101K3RACAUTO:C0402C101K3RACTU
- C78, C92: footprint All Footprints:C75,C78,C92 (3) -> (none)
- C79: renamed from Ct1; footprint All Footprints:C77,C79 (1) -> just-footprints:CAPC10555_55N_KEM; symbol Device:C -> C0603C101K3RACAUTO:C0402C101K3RACTU
- D12: footprint PMEG3005ELD315 -> just-footprints:PMEG3005ELD315
- LED4: footprint All Footprints:LED4 -> (none)
- POT2: footprint All Footprints:POT2 -> just-footprints:SM42TW503; symbol Device:R_Potentiometer -> SM-42TW503:SM-42TW503; Height (none) -> 5.6; Manufacturer_Name (none) -> Nidec Copal; Manufacturer_Part_Number (none) -> SM-42TW503; Mouser Part Number (none) -> 229-SM-42TW503; Mouser Price/Stock (none) -> https://www.mouser.co.uk/ProductDetail/Nidec-Components/SM-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
- R63: footprint RES_PFR05S_CYN -> just-footprints:RES_PFR05S_CYN; symbol 2024-05-10_08-55-23:PFR05S-103-FNH -> PFR05S-103-FNH:PFR05S-103-FNH
- R64: footprint (none) -> just-footprints:RC0402N_PAN; symbol Device:R -> ERJ-2GE0R00X:ERJ-2GE0R00X
- R67, R68, R71: footprint All Footprints:RES_RCA0603_VIS -> just-footprints:RES_RCA0603_VIS; symbol Device:R -> RCA06031K00FKEAHP:RCA06031K00FKEAHP
- R69: footprint All Footprints:ERJP03_PA3__0603_ -> ERJP03_PA3_(0603); symbol Device:R -> ERJ-PA3J100V:ERJ-PA3J100V; Height (none) -> 0.55; Manufacturer_Name (none) -> Panasonic; Manufacturer_Part_Number (none) -> ERJ-PA3J100V; Mouser Part Number (none) -> 667-ERJ-PA3J100V; Mouser Price/Stock (none) -> https://www.mouser.co.uk/ProductDetail/Panasonic/ERJ-PA3J10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
- R70: footprint All Footprints:R70 (1) -> (none)
- R87, R88: footprint All Footprints:RES_ERJUP3_PAN -> (none)
- R89, R90: footprint All Footprints:RESC1508X50N -> (none)
Connections:
- net +5V: now also R67.2, R69.2; no longer R67.1, R69.1, R71.1
- net GND: no longer C77.2, C79.2, C93.2
- net at OP5.1 (OUT), OP5.4 (-IN), TP4.1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: no longer C77.1
- net at C74.1, OP5.3 (+IN), POT2.1 (CCW): now also R67.1; no longer R67.2
- net at C75.1, OP5.5 (V+): now also R69.1; no longer R69.2
- net at R70.2, TP5.1, U11.4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: no longer C79.1, R71.2
- net at R89.2, U13.6 (~{CLR}): no longer C93.1
Other:
- moved on the sheet: D12, R63
