File: TOLT-DC48V-3KW-TOBO2-SinglePhase/Current Comparator & Latch.kicad_sch (KiCad schematic)
At the start: 33 parts, among them Q8 IRLML6346, U11 LMV331, U13 SN74LVC2G74DCUR

Commit message: Commit 1
Parts:
- removed D2 (x2): 500mA/30V/TSLP-2-17, symbol Device:D_Schottky_Filled
- removed R65, R66: 0 0402, symbol Device:R
- C74, C93: value 1uF 25V 0603 -> C0603C105K3RAC7411; footprint (none) -> just-footprints:CAPC17595_95N_KEM; symbol Device:C -> C0603C105K3RAC7411:C0603C105K3RAC7411
- C75, C78, C92: value 0.1uF 25V 0603 -> C0603X104M3RACTU; footprint (none) -> just-footprints:CAPC17795_95N_KEM; symbol Device:C -> C37:C0603X104M3RACTU
- C76: value 1nF 25V 0603 -> C0603X102K3RACAUTO; footprint (none) -> just-footprints:CAPC17795_95N_KEM; symbol Device:C -> C0603X102K3RACAUTO:C0603X102K3RACAUTO
- C77, C79: value 100pF 25V 0603 -> C0402C101K3RACTU; footprint (none) -> just-footprints:CAPC10555_55N_KEM; symbol Device:C -> C0603C101K3RACAUTO:C0402C101K3RACTU
- D12: renamed from D2; value 500mA/30V/TSLP-2-17 -> 500mA/30V/TSLP-2-17
- R63: value 10k 0402 -> PFR05S-103-FNH; footprint (none) -> just-footprints:RES_PFR05S_CYN; symbol Device:R -> PFR05S-103-FNH:PFR05S-103-FNH
- gave numbers to parts that had none: 2
- renumbered TP1 to TP4, TP1 to TP5, TP1 to TP6
Connections:
- net +5V: now also C78.2, C92.2; no longer C78.1, C92.1
- net GND: now also C74.1, C75.1, C76.1, C77.1, C78.1, C79.1, C92.1, C93.1; no longer C74.2, C75.2, C76.2, C77.2, C78.2, C79.2, C92.2, C93.2
- net at OP5.1 (OUT), OP5.4 (-IN), TP4.1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: now also C77.2; no longer C77.1
- net at OP5.3 (+IN), POT2.1, R67.2: now also C74.2; no longer C74.1
- net at OP5.5 (V+), R69.2: now also C75.2; no longer C75.1
- net at D12.1 (K), R63.2, R70.1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: now also C76.2; no longer C76.1
- net at R70.2, R71.2, TP5.1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: now also C79.2; no longer C79.1
- net at R89.2, U13.6 (~{CLR}): now also C93.2; no longer C93.1
Other:
- moved on the sheet: D12, R64
