File: TOLT-DC48V-3KW-TOBO2-SinglePhase/Current Offset.kicad_sch (KiCad schematic)
At the start: 8 parts

Commit message: Commit 1
Parts:
- C72: renamed from C5; value 1uF 25V 0603 -> C0603C105K3RAC7411; footprint (none) -> just-footprints:CAPC17595_95N_KEM; symbol Device:C -> C0603C105K3RAC7411:C0603C105K3RAC7411
- C73: renamed from C5; value 0.1uF 25V 0603 -> C0603X104M3RACTU; footprint (none) -> just-footprints:CAPC17795_95N_KEM; symbol Device:C -> C37:C0603X104M3RACTU
- gave numbers to parts that had none: 5
- renumbered TP1 to TP3
Connections:
- net GND: now also C72.1, C73.1; no longer C72.2, C73.2
- net at OP4.3 (+IN), POT1.1, R60.2: now also C72.2; no longer C72.1
- net at OP4.5 (V+), R62.2: now also C73.2; no longer C73.1
