File: TOLT-DC48V-3KW-TOBO2-SinglePhase/Current amplifier.kicad_sch (KiCad schematic)
At the start: 33 parts

Commit message: Commit 1
Parts:
- removed C5 (x6): 100pF 25V 0603, symbol Device:C
- removed C5 (x2): 0.1uF 25V 0603, symbol Device:C
- removed OP2, OP3: AD8615AUJZ, AD8615AUJZ:SOT95P280X100-5N, symbol AD8615:AD8615AUJZ
- removed R48, R53, R54, R58: 12k 0603, symbol Device:R
- removed R49, R50, R55, R56: 1k 0603, symbol Device:R
- removed R51, R57: 10 0603, symbol Device:R
- removed R52, R59: 10 0402, symbol Device:R
- C60, C62, C63: renamed from C5; value 100pF 25V 0603 -> C0402C101K3RACTU; footprint (none) -> just-footprints:CAPC10555_55N_KEM; symbol Device:C -> C0603C101K3RACAUTO:C0402C101K3RACTU
- C61: renamed from C5; value 0.1uF 25V 0603 -> C0603X104M3RACTU; footprint (none) -> just-footprints:CAPC17795_95N_KEM; symbol Device:C -> C37:C0603X104M3RACTU
Connections:
- net GND: now also C61.1, C63.1; no longer C61.2, C63.2
- net I_SNS_PHASE_U: now also C63.2; no longer C63.1
- net at OP1.1 (OUT), R46.2, R47.1: now also C62.2; no longer C62.1
- net at OP1.4 (-IN), R44.2, R46.1: now also C60.1, C62.1; no longer C60.2, C62.2
- net at OP1.5 (V+), R45.2: now also C61.2; no longer C61.1
- net at OP1.3 (+IN), R42.2, R43.2: now also C60.2; no longer C60.1
Other:
- note removed: "Current Amplifier V Phase"
- note removed: "Current Amplifier W Phase"
- moved on the sheet: OP1, R42, R43, R44, R45, R46, R47
