File: TOLT-DC48V-3KW-TOBO2-SinglePhase/DC-DC Buck Converter.kicad_sch (KiCad schematic)
At the start: 39 parts, among them J3 EXT/ITN 12V, J4 +12V_EXT, J5 +5V_EXT, Q9 FMMT723/SOT, U1 ILD8150XUMA1

Commit message: Commit 1
Parts:
- C1: value 0.1uF 100V 0805 -> C0805X104K1RAC3316; footprint (none) -> just-footprints:C0805; symbol Device:C -> C0805X104K1RAC3316:C0805X104K1RAC3316; Height (none) -> 1.1; Manufacturer_Name (none) -> KEMET; Manufacturer_Part_Number (none) -> C0805X104K1RAC3316
- C10, C11: value 22uF 25V 0805 -> C2012X7S1A226M125AC; footprint (none) -> just-footprints:CAPC2012X145N; symbol Device:C -> C2012X7S1A226M125AC:C2012X7S1A226M125AC; Height (none) -> 1.45; Manufacturer_Name (none) -> TDK; Manufacturer_Part_Number (none) -> C2012X7S1A226M125AC
- C12: value 680pF 25V 0805 -> C0805C681J5RACTU; footprint (none) -> just-footprints:CAPC220145_88N_KEM; symbol Device:C -> C0805X475K3RAC7800:C0805C681J5RACTU; Manufacturer_Name (none) -> KEMET; Manufacturer_Part_Number (none) -> C1206C103J3RACAUTO; Mouser Part Number (none) -> 80-C1206C103J3RAUTO; Mouser Price/Stock (none) -> https://www.mouser.co.uk/ProductDetail/KEMET/C1206C103J3RAC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
- C13: value 0.01uF 25V 1206 -> C1206C103J3RACAUTO; footprint (none) -> just-footprints:C1206; symbol Device:C -> C1206C103J3RACAUTO:C1206C103J3RACAUTO; Manufacturer_Name (none) -> KEMET; Manufacturer_Part_Number (none) -> C1206C103J3RACAUTO; Mouser Part Number (none) -> 80-C1206C103J3RAUTO; Mouser Price/Stock (none) -> https://www.mouser.co.uk/ProductDetail/KEMET/C1206C103J3RAC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
- C14, C16: value 10uF 25V 0805 -> C0805C106M3PACTU; footprint (none) -> just-footprints:CAPC220145_145N_KEM; symbol Device:C -> C0805C106M3PAUTO:C0805C106M3PACTU
- C15, C17: value 0.1uF 25V 0603 -> C0603X104M3RACTU; footprint (none) -> just-footprints:CAPC17795_95N_KEM; symbol Device:C -> C37:C0603X104M3RACTU
- C2: value 4.7nF 100V 0603 -> C0603C103K1RACAUTO; footprint (none) -> just-footprints:C0603; symbol Device:C -> C0603C103K1RACAUTO:C0603C103K1RACAUTO; Height (none) -> 0.87; Manufacturer_Name (none) -> KEMET; Manufacturer_Part_Number (none) -> C0603C103K1RACAUTO; Mouser Part Number (none) -> 80-C0603C103K1RAUTO; Mouser Price/Stock (none) -> https://www.mouser.co.uk/ProductDetail/KEMET/C0603C103K1RAC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
- C3: value 220nF 16V 0603 -> C0603X224J3RACAUTO; footprint (none) -> just-footprints:C0603; symbol Device:C -> C0603X224J3RACAUTO:C0603X224J3RACAUTO; Height (none) -> 0.87; Manufacturer_Name (none) -> KEMET; Manufacturer_Part_Number (none) -> C0603X224J3RACAUTO; Mouser Part Number (none) -> 80-C0603X224J3RAUTO; Mouser Price/Stock (none) -> https://www.mouser.co.uk/ProductDetail/KEMET/C0603X224J3RAC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
- C4: value 100nF 50V 0603 -> C0603C104K5RAC3121; footprint (none) -> just-footprints:CAPC1608X95N; symbol Device:C -> C0603C104K5RAC3121:C0603C104K5RAC3121; Arrow Part Number (none) -> C0603C104K5RAC3121; Arrow Price/Stock (none) -> https://www.arrow.com/en/products/c0603c104k5rac3121/kemet-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; Height (none) -> 0.95; Manufacturer_Name (none) -> KEMET; Manufacturer_Part_Number (none) -> C0603C104K5RAC3121
- C5: value 4.7uF 100V 1210 -> CNA6P1X7R2A475K250AE; footprint (none) -> CAPC3225X280N; symbol Device:C -> CNA6P1X7R2A475K250AE:CNA6P1X7R2A475K250AE; Height (none) -> 2.8; Manufacturer_Name (none) -> TDK; Manufacturer_Part_Number (none) -> CNA6P1X7R2A475K250AE; Mouser Part Number (none) -> 810-CNA6P1X7R2A475K2; Mouser Price/Stock (none) -> https://www.mouser.co.uk/ProductDetail/TDK/CNA6P1X7R2A475K2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
- C6: value 0.1uF 100V 1206 -> C1206F104K1RAC3083; footprint (none) -> just-footprints:CAP_C1206F-RAC-ER_KEM; symbol Device:C -> C1206F104K1RAC3083:C1206F104K1RAC3083
- C7: value 10pF 50V 0603 -> C0603C100K5RACTU; footprint (none) -> just-footprints:C0603; symbol Device:C -> C0603C100K5RACTU:C0603C100K5RACTU; Height (none) -> 0.87; Manufacturer_Name (none) -> KEMET; Manufacturer_Part_Number (none) -> C0603C100K5RACTU; Mouser Part Number (none) -> 80-C0603C100K5R; Mouser Price/Stock (none) -> https://www.mouser.com/Search/Refine.aspx?Keyword=80-C0603C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
- C8: value 100pF 25V 0603 -> C0402C101K3RACTU; footprint (none) -> just-footprints:CAPC10555_55N_KEM; symbol Device:C -> C0603C101K3RACAUTO:C0402C101K3RACTU
- C9: value 4.7uF 25V 0805 -> C0805C681J5RACTU; footprint (none) -> just-footprints:CAPC220145_88N_KEM; symbol Device:C -> C0805X475K3RAC7800:C0805C681J5RACTU
- CR1: renamed from D1; value S210FA -> BAT165E6327HTSA1; footprint (none) -> CR_BAT165_INF; symbol Device:D_Schottky_Filled -> BAT165E6327HTSA1:BAT165E6327HTSA1; Height (none) -> 1.43; Manufacturer_Name (none) -> onsemi; Manufacturer_Part_Number (none) -> S210FA
- D2: footprint (none) -> SODFL3618X143N; symbol Device:D_Schottky_Filled -> S210FA:S210FA; Height (none) -> 1.43; Manufacturer_Name (none) -> onsemi; Manufacturer_Part_Number (none) -> S210FA
- renumbered R3 to R6
Connections:
- net GNDREF: now also C10.1, C11.1, C4.1, C5.1, C6.1, C7.1, C8.1, C9.1; no longer C10.2, C11.2, C4.2, C5.2, C6.2, C7.2, C8.2, C9.2
- net V_BAT+: no longer CR1.2 (A)
- net at U1.3 (DIM): now also C8.2; no longer C8.1
- net at C3.2, R2.2: now also C2.2; no longer C2.1
- net at U1.6 (~{SD}): now also C7.2; no longer C7.1
- net at U1.7 (VCC): now also C4.2; no longer C4.1
- new net: C10.2, C11.2, C2.1, C9.2, J3.01, L1.2, R3.2
- new net: C5.2, C6.2, CR1.2, U1.8 (VIN)
- now unconnected: CR1.1 (K)
