File: TOLT-DC48V-3KW-TOBO2-SinglePhase/Power Board Connector.kicad_sch (KiCad schematic)
At the start: 18 parts, among them J12 Direction Switch, Q7 IRLML6346, U12 PCN10C-32S-2.54DS(72)

Commit message: Commit 1
Parts:
- C80: value 0.1uF 25V 0603 -> C0603X104M3RACTU; footprint (none) -> just-footprints:CAPC17795_95N_KEM; symbol Device:C -> C37:C0603X104M3RACTU
- C81, C82: value 1uF 25V 0603 -> C0603C105K3RAC7411; footprint (none) -> just-footprints:CAPC17595_95N_KEM; symbol Device:C -> C0603C105K3RAC7411:C0603C105K3RAC7411
- renumbered D1 to D15, LED4 to LED3
Connections:
- net BEMF_PHASE_V is gone; now on net U-L: U12. (B9)
- net BEMF_PHASE_W is gone; now on net U-L: U12. (B9)
- net I_SNS_PHASE_V is gone; now on net U-L: U12. (B9)
- net I_SNS_PHASE_W is gone; now on net U-L: U12. (B9)
- net V-H is gone; now on net U-L: U12. (B9)
- net V-L is gone; now on net U-L: U12. (B9)
- net W-H is gone; now on net U-L: U12. (B9)
- net W-L is gone; now on net U-L: U12. (B9)
- net GNDREF: now also C80.1; no longer C80.2
- net GNDS: now also C81.1, C82.1, R80.1; no longer C81.2, C82.2
- net at D15.1 (K), R73.2, R74.1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: now also C80.2; no longer C80.1
- net at R75.1, RT1.1 (V_{DD}): now also C82.2; no longer C82.1
- removed net SD: R80.1, U12. (B9)
- new net: C81.2, R76.1, U12. (B9)
- no-connect marks 12 -> 20
Other:
- moved on the sheet: U12
