File: TOLT-DC48V-3KW-TOBO2-SinglePhase/U-Phase.kicad_sch (KiCad schematic)
At the start: 35 parts, among them Q1 IAUS300N10S5N015TATMA1, Q4 IAUS300N10S5N015TATMA1, U3 2EDL8x24G, U4 NL27WZ08USG

Commit message: Commit 1
Parts:
- C27: value 0.1uF 100V 0805 -> C0805X104K1RAC3316; footprint (none) -> just-footprints:C0805; symbol Device:C -> C0805X104K1RAC3316:C0805X104K1RAC3316; Height (none) -> 1.1; Manufacturer_Name (none) -> KEMET; Manufacturer_Part_Number (none) -> C0805X104K1RAC3316
- C28, C29: value 2.2uF 100V 1206 -> GCM31CC72A225KE02L; footprint (none) -> GCM31CC72A225KE02L:CAPC3216X180N; symbol Device:C -> C28:GCM31CC72A225KE02L
- C30: value 10uF 100V 1210 -> CL32Y106KCVZNWE; footprint (none) -> CAPC3225X280N; symbol Device:C -> CL32Y106KCVZNWE:CL32Y106KCVZNWE; Arrow Part Number (none) -> CL32Y106KCVZNWE; Arrow Price/Stock (none) -> https://www.arrow.com/en/products/cl32y106kcvznwe/samsung-e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; Height (none) -> 2.8; Manufacturer_Name (none) -> SAMSUNG; Manufacturer_Part_Number (none) -> CL32Y106KCVZNWE; Mouser Part Number (none) -> 187-CL32Y106KCVZNWE; Mouser Price/Stock (none) -> https://www.mouser.co.uk/ProductDetail/Samsung-Electro-Mech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
- C31, C32: value 10nF 0603 100V -> CL10B103KC8WPJL; footprint (none) -> just-footprints:CAPC1608X90N; symbol Device:C -> C31:CL10B103KC8WPJL; Height (none) -> 0.9; Manufacturer_Name (none) -> SAMSUNG; Manufacturer_Part_Number (none) -> CL10B103KC8WPJL
- C35: value 0.1uF 50V 1206 -> C1206F104K5RACAUTO; footprint (none) -> just-footprints:C1206; symbol Device:C -> C1206F104K5RACAUTO:C1206F104K5RACAUTO; Manufacturer_Name (none) -> KEMET; Manufacturer_Part_Number (none) -> C1206F104K5RACAUTO; Mouser Part Number (none) -> 80-C1206F104K5RAUTO; Mouser Price/Stock (none) -> https://www.mouser.co.uk/ProductDetail/KEMET/C1206F104K5RAC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
- C36: value 10uF 25V 0603 -> GRM188R61E106MA73J; footprint (none) -> just-footprints:CAPC1608X90N; symbol Device:C -> C33:GRM188R61E106MA73J; Height (none) -> 0.9; Manufacturer_Name (none) -> Murata Electronics; Manufacturer_Part_Number (none) -> GRM188R61E106MA73J; Mouser Part Number (none) -> 81-GRM188R61E106MA3J; Mouser Price/Stock (none) -> https://www.mouser.co.uk/ProductDetail/Murata-Electronics/G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
- C37: value 0.1 uF 25V 0603 -> C0603X104M3RACTU; footprint (none) -> just-footprints:CAPC17795_95N_KEM; symbol Device:C -> C37:C0603X104M3RACTU
- C94: value 4.7uF 100V 2220 -> 22201C475KAT2A; footprint (none) -> 2220_AVX; symbol Device:C -> C94:22201C475KAT2A
- CR4, CR5: renamed from D2; value BAT165E63227HTSAI -> BAT165E6327HTSA1; footprint (none) -> CR_BAT165_INF; symbol Device:D_Schottky_Filled -> BAT165E6327HTSA1:BAT165E6327HTSA1
- D3: renamed from D2; footprint (none) -> SODFL3616X135N; symbol Device:D_Schottky_Filled -> D3:SMD2150PL-TP; Height (none) -> 1.35; Manufacturer_Name (none) -> MCC; Manufacturer_Part_Number (none) -> SMD2150PL-TP; Mouser Part Number (none) -> 833-SMD2150PL-TP; Mouser Price/Stock (none) -> https://www.mouser.co.uk/ProductDetail/Micro-Commercial-Com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
Connections:
- net +5V: now also C37.2; no longer C37.1
- net +BATT: now also C27.2, C28.2, C29.2, C30.2, C94.2; no longer C27.1, C28.1, C29.1, C30.1, C94.1
- net 12V: now also C36.2; no longer C36.1
- net GND: now also C37.1; no longer C37.2
- net GNDREF: now also C27.1, C28.1, C29.1, C30.1, C36.1; no longer C27.2, C28.2, C29.2, C30.2, C36.2
- net U: now also C31.1; no longer C31.2
- net U_CS+: now also C32.1, C94.1; no longer C32.2, C94.2
- net at R15.1: now also C32.2; no longer C32.1
- net at R10.1: now also C31.2; no longer C31.1
