File: EVAL-TOLT-DC-48V-3KW-TOBO2-1206/Current Comparator & Latch.kicad_sch (KiCad schematic)
At the start: 33 parts, among them Q8 IRLML6346, U11 LMV331, U13 SN74LVC2G74DCUR

Commit message: Oct17
Parts:
- C74, C93: value 1uF 25V 0603 -> C1206C105K3RACTM; footprint (none) -> Capacitor-Footprints-1206:C72; symbol Device:C -> C1206C105K3RACTM:C1206C105K3RACTM; Manufacturer_Name (none) -> KEMET; Manufacturer_Part_Number (none) -> C1206C105K3RACTM; Mouser Part Number (none) -> 80-C1206C105K3RACTM; Mouser Price/Stock (none) -> https://www.mouser.co.uk/ProductDetail/KEMET/C1206C105K3RAC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
- C75, C78, C92: value 0.1uF 25V 0603 -> C1206X104M3RECAUTO; footprint (none) -> Capacitor-Footprints-1206:CAPC3316X140N; symbol Device:C -> C1206X104M3RECAUTO:C1206X104M3RECAUTO
- C76: value 1nF 25V 0603 -> C1206C102K3REC; footprint (none) -> Capacitor-Footprints-1206:C76; symbol Device:C -> C1206C102K3REC:C1206C102K3REC
- C77, C79: value 100pF 25V 0603 -> 12063A101KAT2A; footprint (none) -> Capacitor-Footprints-1206:CAP_1206J_AVX; symbol Device:C -> C8:12063A101KAT2A
- D12, D13, D14: renamed from D2; value 500mA/30V/TSLP-2-17 -> 500mA/30V/TSLP-2-17; footprint (none) -> Misc-Footprints-1206:D12
- LED4: footprint (none) -> just-footprints:LED4
- OP5: renamed from OP?; footprint AD8615AUJZ:SOT95P280X100-5N -> infineon-library-footprints:AD8615
- POT2: renamed from RV?; footprint (none) -> just-footprints:POT2
- Q8: footprint Package_TO_SOT_SMD:SOT-23 -> just-footprints:Q8 (1)
- R63: footprint (none) -> Resistor-Footprint:R63
- R64, R65, R66: footprint (none) -> Resistor-Footprint:R64
- R67: footprint (none) -> Resistor-Footprint:R67
- R68: footprint (none) -> Resistor-Footprint:R68
- R69: footprint (none) -> Resistor-Footprint:R12
- R70: footprint (none) -> Resistor-Footprint:R70
- R71: footprint (none) -> Resistor-Footprint:R71
- R87: footprint (none) -> Resistor-Footprint:R43
- U11: footprint (none) -> infineon-library-footprints:LMV331M5
- U13: footprint SN74LVC2G74DCUR:SOP50P310X90-8N -> infineon-library-footprints:SN74LVC2G74DCUR
- renumbered TP1 to TP4, TP1 to TP5, TP1 to TP6
Connections:
- net +5V: now also C78.2, C92.2; no longer C78.1, C92.1
- net GND: now also C74.1, C75.1, C76.1, C77.1, C78.1, C79.1, C92.1, C93.1; no longer C74.2, C75.2, C76.2, C77.2, C78.2, C79.2, C92.2, C93.2
- net at OP5.1 (OUT), OP5.4 (-IN), TP4.1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: now also C77.2; no longer C77.1
- net at OP5.3 (+IN), POT2.1, R67.2: now also C74.2; no longer C74.1
- net at OP5.5 (V+), R69.2: now also C75.2; no longer C75.1
- net at D12.1 (K), D13.1 (K), D14.1 (K)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: now also C76.2; no longer C76.1
- net at R70.2, R71.2, TP5.1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: now also C79.2; no longer C79.1
- net at R89.2, U13.6 (~{CLR}): now also C93.2; no longer C93.1
Other:
- moved on the sheet: R69
