File: EVAL-TOLT-DC-48V-3KW-TOBO2-1206/Current Offset.kicad_sch (KiCad schematic)
At the start: 8 parts

Commit message: Oct17
Parts:
- C72: renamed from C5; value 1uF 25V 0603 -> C1206C105K3RACTM; footprint (none) -> Capacitor-Footprints-1206:C72; symbol Device:C -> C1206C105K3RACTM:C1206C105K3RACTM; Manufacturer_Name (none) -> KEMET; Manufacturer_Part_Number (none) -> C1206C105K3RACTM; Mouser Part Number (none) -> 80-C1206C105K3RACTM; Mouser Price/Stock (none) -> https://www.mouser.co.uk/ProductDetail/KEMET/C1206C105K3RAC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
- C73: renamed from C5; value 0.1uF 25V 0603 -> C1206X104M3RECAUTO; footprint (none) -> Capacitor-Footprints-1206:CAPC3316X140N; symbol Device:C -> C1206X104M3RECAUTO:C1206X104M3RECAUTO
- OP4: renamed from OP?; footprint AD8615AUJZ:SOT95P280X100-5N -> infineon-library-footprints:AD8615
- POT1: renamed from RV?; footprint (none) -> just-footprints:POT2
- R60: renamed from R?; footprint (none) -> Resistor-Footprint:R60
- R61: renamed from R?; footprint (none) -> Resistor-Footprint:R61
- R62: renamed from R?; footprint (none) -> Resistor-Footprint:R12
- renumbered TP1 to TP3
Connections:
- net GND: now also C72.1, C73.1; no longer C72.2, C73.2
- net at OP4.3 (+IN), POT1.1, R60.2: now also C72.2; no longer C72.1
- net at OP4.5 (V+), R62.2: now also C73.2; no longer C73.1
