File: EVAL-TOLT-DC-48V-3KW-TOBO2-1206/Current amplifier.kicad_sch (KiCad schematic)
At the start: 33 parts

Commit message: Oct17
Parts:
- removed C5 (x6): 100pF 25V 0603, symbol Device:C
- removed C5 (x2): 0.1uF 25V 0603, symbol Device:C
- removed OP2, OP3: AD8615AUJZ, AD8615AUJZ:SOT95P280X100-5N, symbol AD8615:AD8615AUJZ
- removed R48, R53, R54, R58: 12k 0603, symbol Device:R
- removed R49, R50, R55, R56: 1k 0603, symbol Device:R
- removed R51, R57: 10 0603, symbol Device:R
- removed R52, R59: 10 0402, symbol Device:R
- C60, C63: renamed from C5; value 100pF 25V 0603 -> 12063A101KAT2A; footprint (none) -> Capacitor-Footprints-1206:CAP_1206J_AVX; symbol Device:C -> C8:12063A101KAT2A
- C61: renamed from C5; value 0.1uF 25V 0603 -> C1206X104M3RECAUTO; footprint (none) -> Capacitor-Footprints-1206:CAPC3316X140N; symbol Device:C -> C1206X104M3RECAUTO:C1206X104M3RECAUTO
- C62: renamed from C5; value 100pF 25V 0603 -> C5750X7R2A475K230KA; footprint (none) -> Capacitor-Footprints-1206:CAP_1206J_AVX; symbol Device:C -> C5750X7R2A475K230KA:C5750X7R2A475K230KA; Height (none) -> 2.5; Manufacturer_Name (none) -> TDK; Manufacturer_Part_Number (none) -> C5750X7R2A475K230KA; Mouser Part Number (none) -> 810-C5750X7R2A475K; Mouser Price/Stock (none) -> https://www.mouser.co.uk/ProductDetail/TDK/C5750X7R2A475K23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
- OP1: footprint AD8615AUJZ:SOT95P280X100-5N -> infineon-library-footprints:AD8615
- R42, R46: footprint (none) -> Resistor-Footprint:R42
- R43, R44: footprint (none) -> Resistor-Footprint:R43
- R45: footprint (none) -> Resistor-Footprint:R12
- R47: footprint (none) -> Resistor-Footprint:R47
Connections:
- net GND: now also C61.1, C63.1; no longer C61.2, C63.2
- net I_SNS_PHASE_U: now also C63.2; no longer C63.1
- net at OP1.1 (OUT), R46.2, R47.1: now also C62.2; no longer C62.1
- net at OP1.4 (-IN), R44.2, R46.1: now also C60.1, C62.1; no longer C60.2, C62.2
- net at OP1.5 (V+), R45.2: now also C61.2; no longer C61.1
- net at OP1.3 (+IN), R42.2, R43.2: now also C60.2; no longer C60.1
Other:
- note removed: "Current Amplifier V Phase"
- note removed: "Current Amplifier W Phase"
- moved on the sheet: OP1, R42, R43, R44, R45, R46, R47
