File: EVAL-TOLT-DC-48V-3KW-TOBO2-1206/DC-DC Buck Converter.kicad_sch (KiCad schematic)
At the start: 39 parts, among them J3 EXT/ITN 12V, J4 +12V_EXT, J5 +5V_EXT, Q9 FMMT723/SOT, U1 ILD8150XUMA1

Commit message: Oct17
Parts:
- C1: value 0.1uF 100V 0805 -> C1206F104K1RACAUTO; footprint (none) -> Capacitor-Footprints-1206:C1; symbol Device:C -> C1206F104K1RACAUTO:C1206F104K1RACAUTO; Manufacturer_Name (none) -> KEMET; Manufacturer_Part_Number (none) -> C1206F104K1RACAUTO; Mouser Part Number (none) -> 80-C1206F104K1RAUTO; Mouser Price/Stock (none) -> https://www.mouser.co.uk/ProductDetail/KEMET/C1206F104K1RAC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
- C10, C11: value 22uF 25V 0805 -> C1206C226M8RAC7800; footprint (none) -> Capacitor-Footprints-1206:CAPC340180_180N_KEM; symbol Device:C -> C10:C1206C226M8RAC7800
- C12: value 680pF 25V 0805 -> C1206C681J5RACTU; footprint (none) -> Capacitor-Footprints-1206:C12; symbol Device:C -> C1206C681J5RACTU:C1206C681J5RACTU; Manufacturer_Name (none) -> KEMET; Manufacturer_Part_Number (none) -> C1206C681J5RACTU; Mouser Part Number (none) -> 80-C1206C681J5RACTU; Mouser Price/Stock (none) -> https://www.mouser.co.uk/ProductDetail/KEMET/C1206C681J5RAC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
- C13: value 0.01uF 25V 1206 -> C1206C103J3RACAUTO; footprint (none) -> Capacitor-Footprints-1206:C13; symbol Device:C -> C1206C103J3RACAUTO:C1206C103J3RACAUTO; Manufacturer_Name (none) -> KEMET; Manufacturer_Part_Number (none) -> C1206C103J3RACAUTO; Mouser Part Number (none) -> 80-C1206C103J3RAUTO; Mouser Price/Stock (none) -> https://www.mouser.co.uk/ProductDetail/KEMET/C1206C103J3RAC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
- C14, C16: value 10uF 25V 0805 -> C1206C106M3PACTU; footprint (none) -> Capacitor-Footprints-1206:C14; symbol Device:C -> C1206C106M3PACTU:C1206C106M3PACTU; Manufacturer_Name (none) -> KEMET; Manufacturer_Part_Number (none) -> C1206C106M3PACTU; Mouser Part Number (none) -> 80-C1206C106M3P; Mouser Price/Stock (none) -> https://www.mouser.co.uk/ProductDetail/KEMET/C1206C106M3PAC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
- C15, C17: value 0.1uF 25V 0603 -> C1206X104M3RECAUTO; footprint (none) -> Capacitor-Footprints-1206:CAPC3316X140N; symbol Device:C -> C1206X104M3RECAUTO:C1206X104M3RECAUTO
- C2: value 4.7nF 100V 0603 -> C1206C472K1RACTU; footprint (none) -> Capacitor-Footprints-1206:C2; symbol Device:C -> C1206C472K1RACTU:C1206C472K1RACTU; Manufacturer_Name (none) -> KEMET; Manufacturer_Part_Number (none) -> C1206C472K1RACTU; Mouser Part Number (none) -> 80-C1206C472K1R; Mouser Price/Stock (none) -> https://www.mouser.co.uk/ProductDetail/KEMET/C1206C472K1RAC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
- C3: value 220nF 16V 0603 -> 12063C224JAT2A; footprint (none) -> Capacitor-Footprints-1206:CAPC3216X94N; symbol Device:C -> 12063C224JAT2A:12063C224JAT2A; Manufacturer_Name (none) -> Kyocera AVX; Manufacturer_Part_Number (none) -> 12063C224JAT2A; Mouser Part Number (none) -> 581-12063C224JAT2A
- C4: value 100nF 50V 0603 -> C1206C104K5RAC; footprint (none) -> Capacitor-Footprints-1206:CAPC3216X88N; symbol Device:C -> C1206C104K5RAC:C1206C104K5RAC; Arrow Part Number (none) -> C1206C104K5RAC; Arrow Price/Stock (none) -> https://www.arrow.com/en/products/c1206c104k5rac/kemet-corp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; Height (none) -> 0.88; Manufacturer_Name (none) -> KEMET; Manufacturer_Part_Number (none) -> C1206C104K5RAC; Mouser Part Number (none) -> 80-C1206C104K5RAC; Mouser Price/Stock (none) -> https://www.mouser.co.uk/ProductDetail/KEMET/C1206C104K5RAC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
- C5: value 4.7uF 100V 1210 -> CNA6P1X7R2A475K250AE; footprint (none) -> Capacitor-Footprints-1206:CAPC3225X280N; symbol Device:C -> CNA6P1X7R2A475K250AE:CNA6P1X7R2A475K250AE; Arrow Part Number (none) -> CNA6P1X7R2A475K250AE; Arrow Price/Stock (none) -> https://www.arrow.com/en/products/cna6p1x7r2a475k250ae/tdk?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; Height (none) -> 2.8; Manufacturer_Name (none) -> TDK; Manufacturer_Part_Number (none) -> CNA6P1X7R2A475K250AE; Mouser Part Number (none) -> 810-CNA6P1X7R2A475K2; Mouser Price/Stock (none) -> https://www.mouser.co.uk/ProductDetail/TDK/CNA6P1X7R2A475K2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
- C6: value 0.1uF 100V 1206 -> C1206F104K1RACAUTO; footprint (none) -> Capacitor-Footprints-1206:C6; symbol Device:C -> C1206F104K1RACAUTO:C1206F104K1RACAUTO; Manufacturer_Name (none) -> KEMET; Manufacturer_Part_Number (none) -> C1206F104K1RACAUTO; Mouser Part Number (none) -> 80-C1206F104K1RAUTO; Mouser Price/Stock (none) -> https://www.mouser.co.uk/ProductDetail/KEMET/C1206F104K1RAC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
- C7: value 10pF 50V 0603 -> C1206X104M3RECAUTO; footprint (none) -> Capacitor-Footprints-1206:C7; symbol Device:C -> C1206X104M3RECAUTO:C1206X104M3RECAUTO; Height (none) -> 0.88; Manufacturer_Name (none) -> KEMET; Manufacturer_Part_Number (none) -> C1206C100K5RACAUTO; Mouser Part Number (none) -> 80-C1206C100K5RAUTO; Mouser Price/Stock (none) -> https://www.mouser.co.uk/ProductDetail/KEMET/C1206C100K5RAC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
- C8: value 100pF 25V 0603 -> 1206Y0250101KXT; footprint (none) -> Capacitor-Footprints-1206:CAP_1206J_AVX; symbol Device:C -> 1206Y0250101KXT:1206Y0250101KXT
- C9: value 4.7uF 25V 0805 -> C1206C475K3RAC7800; footprint (none) -> Capacitor-Footprints-1206:C9; symbol Device:C -> C9:C1206C475K3RAC7800
- D1, D2: footprint (none) -> Misc-Footprints-1206:D1; symbol Device:D_Schottky_Filled -> D1:S210FA; Height (none) -> 1.43; Manufacturer_Name (none) -> onsemi; Manufacturer_Part_Number (none) -> S210FA; Mouser Part Number (none) -> 512-S210FA; Mouser Price/Stock (none) -> https://www.mouser.co.uk/ProductDetail/onsemi-Fairchild/S21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
- G1, R1: footprint (none) -> Resistor-Footprint:R1
- J3: footprint TSW-103-08-L-S:SAMTEC_TSW-103-08-L-S -> Resistor-Footprint:R2
- J4: footprint 1725656 -> Resistor-Footprint:R3
- J5: footprint 1725656 -> Resistor-Footprint:R4
- L1: footprint (none) -> Resistor-Footprint:R6
- LED1, LED2: footprint (none) -> just-footprints:LEDC1608X80N
- Q9: footprint Package_TO_SOT_SMD:SOT-23 -> infineon-library-footprints:LMV331M5
- R2: footprint (none) -> Resistor-Footprint:R2
- R3: footprint (none) -> Resistor-Footprint:R3
- R4: footprint (none) -> Resistor-Footprint:R4
- R5: footprint (none) -> Resistor-Footprint:R5
- R6: renamed from R3; footprint (none) -> Resistor-Footprint:R6
- R8: footprint (none) -> Resistor-Footprint:R8
- U1: footprint ILD8150XUMA1:SOIC127P600X175-8N -> infineon-library-footprints:ILD8150
Connections:
- net GNDREF: now also C10.1, C11.1, C4.1, C5.1, C6.1, C7.1, C8.1, C9.1; no longer C10.2, C11.2, C4.2, C5.2, C6.2, C7.2, C8.2, C9.2
- net at C2.2, J3.01, L1.2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: now also C10.2, C11.2, C9.2; no longer C10.1, C11.1, C9.1
- net at U1.3 (DIM): now also C8.2; no longer C8.1
- net at U1.6 (~{SD}): now also C7.2; no longer C7.1
- net at U1.7 (VCC): now also C4.2; no longer C4.1
- net at D1.1 (K), U1.8 (VIN): now also C5.2, C6.2; no longer C5.1, C6.1
