File: EVAL-TOLT-DC-48V-3KW-TOBO2-1206/Power Board Connector.kicad_sch (KiCad schematic)
At the start: 18 parts, among them J12 Direction Switch, Q7 IRLML6346, U12 PCN10C-32S-2.54DS(72)

Commit message: Oct17
Parts:
- C80: value 0.1uF 25V 0603 -> C1206X104M3RECAUTO; footprint (none) -> Capacitor-Footprints-1206:CAPC3316X140N; symbol Device:C -> C1206X104M3RECAUTO:C1206X104M3RECAUTO
- C81, C82: value 1uF 25V 0603 -> C1206C105K3RACTM; footprint (none) -> Capacitor-Footprints-1206:C72; symbol Device:C -> C1206C105K3RACTM:C1206C105K3RACTM; Manufacturer_Name (none) -> KEMET; Manufacturer_Part_Number (none) -> C1206C105K3RACTM; Mouser Part Number (none) -> 80-C1206C105K3RACTM; Mouser Price/Stock (none) -> https://www.mouser.co.uk/ProductDetail/KEMET/C1206C105K3RAC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
- D15: renamed from D1; footprint (none) -> Misc-Footprints-1206:D15
- J12: footprint TSW-102-08-L-S:SAMTEC_TSW-102-08-L-S -> Resistor-Footprint:R5
- LED3: renamed from LED4; footprint (none) -> just-footprints:LEDC1608X80N
- Q7: footprint Package_TO_SOT_SMD:SOT-23 -> just-footprints:Q8 (1)
- R72: footprint (none) -> Resistor-Footprint:R72
- R73: footprint (none) -> Resistor-Footprint:R73
- R80: footprint (none) -> Resistor-Footprint:R7
- RT1: footprint Package_TO_SOT_SMD:SOT-23 -> infineon-library-footprints:MCP9700AT_E_TT
Connections:
- net GNDREF: now also C80.1; no longer C80.2
- net GNDS: now also C81.1, C82.1; no longer C81.2, C82.2
- net at D15.1 (K), R73.2, R74.1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: now also C80.2; no longer C80.1
- net at R75.1, RT1.1 (V_{DD}): now also C82.2; no longer C82.1
- new net: C81.2, R76.1, U12. (B9)
