File: EVAL-TOLT-DC-48V-3KW-TOBO2-1206/U-Phase.kicad_sch (KiCad schematic)
At the start: 35 parts, among them Q1 IAUS300N10S5N015TATMA1, Q4 IAUS300N10S5N015TATMA1, U3 2EDL8x24G, U4 NL27WZ08USG

Commit message: Oct17
Parts:
- C27: value 0.1uF 100V 0805 -> C1206C104K5RACAUTO; footprint (none) -> Capacitor-Footprints-1206:C1; symbol Device:C -> C1206C104K5RACAUTO:C1206C104K5RACAUTO; Manufacturer_Name (none) -> KEMET; Manufacturer_Part_Number (none) -> C1206C104K5RACAUTO; Mouser Part Number (none) -> 80-C1206C104K5RAUTO; Mouser Price/Stock (none) -> https://www.mouser.co.uk/ProductDetail/KEMET/C1206C104K5RAC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
- C28, C29: value 2.2uF 100V 1206 -> C3216X7S2A225K160AB; footprint (none) -> Capacitor-Footprints-1206:CAP_3216_TDK; symbol Device:C -> C28:C3216X7S2A225K160AB
- C30: value 10uF 100V 1210 -> GRM32EC72A106KE05L; footprint (none) -> Capacitor-Footprints-1206:CAPC3225X270N; symbol Device:C -> GRM32EC72A106KE05L:GRM32EC72A106KE05L
- C31, C32: value 10nF 0603 100V -> C1206X103K1RECAUTO; footprint (none) -> Capacitor-Footprints-1206:CAPC3316X98N; symbol Device:C -> C1206X103K1RECAUTO:C1206X103K1RECAUTO
- C33, C34: value opt/0603/25V -> CC1206KFX7R8BB105; footprint (none) -> Capacitor-Footprints-1206:CAP_CC1206_YAG; symbol Device:C -> C33:CC1206KFX7R8BB105
- C35: value 0.1uF 50V 1206 -> C1206C104K5RAC7025; footprint (none) -> Capacitor-Footprints-1206:CAPC340180_88N_KEM; symbol Device:C -> C35:C1206C104K5RAC7025
- C36: value 10uF 25V 0603 -> TMK316BJ106ML-T; footprint (none) -> Capacitor-Footprints-1206:CAP_TMK316AB7475KL-T_TAY; symbol Device:C -> C36:TMK316BJ106ML-T
- C37: value 0.1 uF 25V 0603 -> C1206X104M3RECAUTO; footprint (none) -> Capacitor-Footprints-1206:CAPC3316X140N; symbol Device:C -> C1206X104M3RECAUTO:C1206X104M3RECAUTO
- C83, C84: value 100pf 25V 0402 -> 1206Y0250101KXT; footprint (none) -> Capacitor-Footprints-1206:CAPC3216X160N; symbol Device:C -> 1206Y0250101KXT:1206Y0250101KXT
- C94: value 4.7uF 100V 2220 -> C5750X7R2A475K230KA; footprint (none) -> Capacitor-Footprints-1206:CAPC3216X160N; symbol Device:C -> C5750X7R2A475K230KA:C5750X7R2A475K230KA; Height (none) -> 2.5; Manufacturer_Name (none) -> TDK; Manufacturer_Part_Number (none) -> C5750X7R2A475K230KA; Mouser Part Number (none) -> 810-C5750X7R2A475K; Mouser Price/Stock (none) -> https://www.mouser.co.uk/ProductDetail/TDK/C5750X7R2A475K23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
- D3: renamed from D2; footprint (none) -> Misc-Footprints-1206:D3
- D4, D5: renamed from D2; footprint (none) -> Misc-Footprints-1206:D4
- Q1: footprint PG-HDSOP-16-2 -> just-footprints:Q1
- Q4: footprint PG-HDSOP-16-2 -> just-footprints:Q4
- R10, R15: footprint (none) -> Resistor-Footprint:R10
- R11, R16: footprint (none) -> Resistor-Footprint:R11
- R12, R18: footprint (none) -> Resistor-Footprint:R12
- R13, R19: footprint (none) -> Resistor-Footprint:R13
- R14: footprint (none) -> Resistor-Footprint:R14
- R17: footprint (none) -> Resistor-Footprint:R17
- R81, R82: footprint (none) -> just-footprints:R81
- RS1: footprint (none) -> just-footprints:RES_HCS3920_1L00_STP
- U3: footprint (none) -> just-footprints:U3
- U4: footprint NL27WZ08USG:SOP50P310X90-8N -> just-footprints:U4
Connections:
- net +5V: now also C37.2; no longer C37.1
- net +BATT: now also C27.2, C28.2, C29.2, C30.2, C94.2; no longer C27.1, C28.1, C29.1, C30.1, C94.1
- net 12V: now also C36.2; no longer C36.1
- net GND: now also C37.1, C83.1, C84.1; no longer C37.2, C83.2, C84.2
- net GNDREF: now also C27.1, C28.1, C29.1, C30.1, C36.1; no longer C27.2, C28.2, C29.2, C30.2, C36.2
- net U: now also C31.1, C33.1, C35.1; no longer C31.2, C33.2, C35.2
- net U-HIN: now also C83.2; no longer C83.1
- net U-LIN: now also C84.2; no longer C84.1
- net U_CS+: now also C32.1, C34.1, C94.1; no longer C32.2, C34.2, C94.2
- net at D3.1 (K), U3.2 (HB): now also C35.2; no longer C35.1
- net at D5.2 (A), Q4.8 (GATE), R16.2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: now also C34.2; no longer C34.1
- net at R15.1: now also C32.2; no longer C32.1
- net at D4.2 (A), Q1.8 (GATE), R11.2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: now also C33.2; no longer C33.1
- net at R10.1: now also C31.2; no longer C31.1
Other:
- moved on the sheet: R15
