File: EVAL-TOLT-DC-48V-3KW-TOBO2-1206/W-Phase.kicad_sch (KiCad schematic)
At the start: 35 parts, among them Q1 IAUS300N10S5N015TATMA1, Q4 IAUS300N10S5N015TATMA1, U3 2EDL8x24G, U4 NL27WZ08USG

Commit message: Oct17
Parts:
- renumbered C32 to C?, C36 to C?, C31 to C?, C94 to C?, C84 to C?, C35 to C?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
