File: EVAL-TOLT-DC48V-3KW-TOBO2-1206/EVAL_TOLT_DC48V_3KW.kicad_pcb (KiCad board)
At the start: 4 copper layers, 170 x 120 mm, 146 parts, among them IC1 LM5013QDDARQ1, J1 V_BAT+, J12 Direction Switch, J2 V_BAT-, J5 +5V_EXT, J6 MountingHole_3.2mm_M3_DIN965, J7 MountingHole_3.2mm_M3_DIN965, J8 MountingHole_3.2mm_M3_DIN965, J9 MountingHole_3.2mm_M3_DIN965, Q1 IAUS300N10S5N015TATMA1, Q4 IAUS300N10S5N015TATMA1, Q7 IRLML6346, Q8 IRLML6346, U11 LMV331, U12 PCN10-32S-2.54DSA72, U13 SN74LVC2G74DCUR, U3 2EDL8x24G, U4 NL27WZ08USG

Commit message: v01112024
New PCB Version for Zones
Parts:
- removed J6, J7, J8, J9: MountingHole_3.2mm_M3_DIN965, MountingHole:MountingHole_3.2mm_M3_DIN965
- added G***: LOGO, 1206-Infineon-Library:Aryan-Pepe-Logo, F.Cu at (227.5, 132.5)
- added REF**: MountingHole_3.2mm_M3_DIN965, MountingHole:MountingHole_3.2mm_M3_DIN965, F.Cu at (245.0, 35.0)
- added REF**: MountingHole_3.2mm_M3_DIN965, MountingHole:MountingHole_3.2mm_M3_DIN965, F.Cu at (245.0, 145.0)
- added REF**: MountingHole_3.2mm_M3_DIN965, MountingHole:MountingHole_3.2mm_M3_DIN965, F.Cu at (85.0, 145.0)
- added REF**: MountingHole_3.2mm_M3_DIN965, MountingHole:MountingHole_3.2mm_M3_DIN965, F.Cu at (85.0, 35.0)
- C13, C14, C15, C16, C17, C20, C21, C22, C23, C24, C25, C26, C27, C28, C29, C30, C31, C32, C35, C36, C37, C506, C507, C508, C60, C61, C62, C63, C72, C73, C74, C75, C76, C77, C78, C79, C80, C81, C811, C82, C821, C83, C84, C89, C92, C93, C94, D12, D15, D3, D4, D5, G1, IC1, L1, OP1, OP4, OP5, Q7, Q8, R1, R10, R11, R12, R13, R15, R16, R18, R19, R4, R42, R43, R44, R45, R46, R47, R501, R502, R503, R60, R61, R62, R63, R64, R67, R68, R69, R70, R71, R72, R73, R74, R75, R751, R76, R762, R77, R78, R79, R8, R80, R81, R82, R87, R88, R89, R90, RS1, RT1, RT2, U11, U13, U3, U4: moved to F.Cu
- moved R47 344.3 mm to (-95.1, 66.1)
- moved C81 330.6 mm to (-70.7, 1.08)
- moved C19 329.2 mm to (-132.5, 18.5)
- moved R76 317.2 mm to (-58.6, 6.76), turned to 0 degrees
- moved R7 314.7 mm to (-94.9, 62.7), turned to 0 degrees
- moved C18 311.8 mm to (-132.5, -1.57)
- moved R72 308.7 mm to (-76.9, 0.39), turned to 0 degrees
- moved R74 308.4 mm to (-76.9, 3.65), turned to 0 degrees
- moved C98 306.2 mm to (-132.5, 58.5), turned to 0 degrees
- moved C22 300.1 mm to (-94.8, 32.3), turned to 0 degrees
- moved C21 298.4 mm to (-94.8, 27.9), turned to 0 degrees
- moved C89 297.9 mm to (-88.9, 32.3), turned to 0 degrees
- moved R78 297.0 mm to (-76.9, 10.2), turned to 0 degrees
- moved R79 296.9 mm to (-76.9, 13.4), turned to 0 degrees
- moved C20 296.5 mm to (-94.8, 23.4), turned to 0 degrees
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Connections:
- C18 pad 2: Net-(J1-Pin_1) -> V_BAT+
- C19 pad 2: Net-(J1-Pin_1) -> V_BAT+
- C20 pad 2: Net-(J1-Pin_1) -> V_BAT+
- C21 pad 2: Net-(J1-Pin_1) -> V_BAT+
- C22 pad 2: Net-(J1-Pin_1) -> V_BAT+
- C23 pad 2: Net-(J1-Pin_1) -> V_BAT+
- C24 pad 2: Net-(J1-Pin_1) -> V_BAT+
- C25 pad 2: Net-(J1-Pin_1) -> V_BAT+
- C26 pad 2: Net-(J1-Pin_1) -> V_BAT+
- C89 pad 2: Net-(J1-Pin_1) -> V_BAT+
- C97 pad 2: Net-(J1-Pin_1) -> V_BAT+
- C98 pad 2: Net-(J1-Pin_1) -> V_BAT+
- C99 pad 2: Net-(J1-Pin_1) -> V_BAT+
- J1 pad 1: Net-(J1-Pin_1) -> V_BAT+
Routing:
- net Net-(OP1--IN): track 2.10 -> 0.00 mm
- added copper zone on In2.Cu, net /U-Phase/+5V
- added copper zone on In2.Cu, net /U-Phase/12V
- added copper zone on In2.Cu, net /U-Phase/U
- added copper zone on In2.Cu, net /U-Phase/U_CS+
- added copper zone on In3.Cu, net 5V
- added copper zone on In4.Cu, net GNDS
- added copper zone on In2.Cu, net V_BAT+
- added copper zone on In2.Cu, net V_BAT-
Other:
- copper layers 4 -> 6

Commit message: v06112024
Parts:
- removed G***: LOGO, 1206-Infineon-Library:Aryan-Pepe-Logo
- added J3: EXT/ITN 12V, infineon-library-footprints:TSW-103-08-L-S, F.Cu at (116.5, 136.1)
- added J4: +12V_EXT, Misc-Footprints:J4, F.Cu at (113.0, 145.5)
- C13: footprint Kap-1206-Footprints:C13 -> Capacitor_SMD:C_1206_3216Metric
- C14, C16: footprint Kap-1206-Footprints:C14 -> Capacitor_SMD:C_1206_3216Metric
- C15, C17, C37, C61, C73, C75, C78, C80, C92: footprint Kap-1206-Footprints:C15 -> Capacitor_SMD:C_1206_3216Metric
- C20, C21, C22, C23, C24, C25, C26, C89: footprint Kap-1206-Footprints:C20 -> Capacitor_SMD:C_1206_3216Metric
- C27: footprint Kap-1206-Footprints:C1 -> Capacitor_SMD:C_1206_3216Metric
- C28, C29: footprint Kap-1206-Footprints:C28 -> Capacitor_SMD:C_1206_3216Metric
- C30: footprint Kap-1206-Footprints:C30 -> Capacitor_SMD:C_1206_3216Metric
- C31, C32: footprint Kap-1206-Footprints:C31 -> Capacitor_SMD:C_1206_3216Metric
- C35: footprint Kap-1206-Footprints:C35 -> Capacitor_SMD:C_1206_3216Metric
- C36: footprint Kap-1206-Footprints:C36 -> Capacitor_SMD:C_1206_3216Metric
- C506, C507: footprint Kap-1206-Footprints:C506 -> Capacitor_SMD:C_1206_3216Metric
- C508: footprint Kap-1206-Footprints:C508 -> Capacitor_SMD:C_1206_3216Metric
- C60, C62, C63, C77, C79: footprint Kap-1206-Footprints:C8 -> Capacitor_SMD:C_1206_3216Metric
- C72, C74, C81, C811, C82, C821, C93: footprint Kap-1206-Footprints:C72 -> Capacitor_SMD:C_1206_3216Metric
- C76: footprint Kap-1206-Footprints:C76 -> Capacitor_SMD:C_1206_3216Metric
- C83, C84: footprint Kap-1206-Footprints:C83 -> Capacitor_SMD:C_1206_3216Metric
- C94: footprint Kap-1206-Footprints:C94 -> Capacitor_SMD:C_1206_3216Metric
- R1: footprint Resistor-1206-Footprints:R1 -> Resistor_SMD:R_1206_3216Metric_Pad1.30x1.75mm_HandSolder
- R10, R15: footprint Resistor-1206-Footprints:R10 -> Resistor_SMD:R_1206_3216Metric_Pad1.30x1.75mm_HandSolder
- R11, R16: footprint Resistor-1206-Footprints:R11 -> Resistor_SMD:R_1206_3216Metric_Pad1.30x1.75mm_HandSolder
- R12, R18, R45, R62, R69: footprint Resistor-1206-Footprints:R12 -> Resistor_SMD:R_1206_3216Metric_Pad1.30x1.75mm_HandSolder
- R13, R19, R73: footprint Resistor-1206-Footprints:R13 -> Resistor_SMD:R_1206_3216Metric_Pad1.30x1.75mm_HandSolder
- R14: footprint Resistor-1206-Footprints:R14 -> Resistor_SMD:R_1206_3216Metric_Pad1.30x1.75mm_HandSolder
- R17: footprint Resistor-1206-Footprints:R17 -> Resistor_SMD:R_1206_3216Metric_Pad1.30x1.75mm_HandSolder
- R4: footprint Resistor-1206-Footprints:R4 -> Resistor_SMD:R_1206_3216Metric_Pad1.30x1.75mm_HandSolder
- R42, R46: footprint Resistor-1206-Footprints:R42 -> Resistor_SMD:R_1206_3216Metric_Pad1.30x1.75mm_HandSolder
- R43, R44: footprint Resistor-1206-Footprints:R43 -> Resistor_SMD:R_1206_3216Metric_Pad1.30x1.75mm_HandSolder
- R47, R81, R82: footprint Resistor-1206-Footprints:R47 -> Resistor_SMD:R_1206_3216Metric_Pad1.30x1.75mm_HandSolder
- R501: footprint Resistor-1206-Footprints:R501 -> Resistor_SMD:R_1206_3216Metric_Pad1.30x1.75mm_HandSolder
- R502: footprint Resistor-1206-Footprints:R502 -> Resistor_SMD:R_1206_3216Metric_Pad1.30x1.75mm_HandSolder
- R503: footprint Resistor-1206-Footprints:R503 -> Resistor_SMD:R_1206_3216Metric_Pad1.30x1.75mm_HandSolder
- R60: footprint Resistor-1206-Footprints:R60 -> Resistor_SMD:R_1206_3216Metric_Pad1.30x1.75mm_HandSolder
- R61, R67, R68, R71: footprint Resistor-1206-Footprints:R61 -> Resistor_SMD:R_1206_3216Metric_Pad1.30x1.75mm_HandSolder
- R63: footprint Resistor-1206-Footprints:R63 -> Resistor_SMD:R_1206_3216Metric_Pad1.30x1.75mm_HandSolder
- R64: footprint Resistor-1206-Footprints:R64 -> Resistor_SMD:R_1206_3216Metric_Pad1.30x1.75mm_HandSolder
- R7, R80: footprint Resistor-1206-Footprints:R7 -> Resistor_SMD:R_1206_3216Metric_Pad1.30x1.75mm_HandSolder
- R70: footprint Resistor-1206-Footprints:R70 -> Resistor_SMD:R_1206_3216Metric_Pad1.30x1.75mm_HandSolder
- R72, R78, R79, R87, R88: footprint Resistor-1206-Footprints:R72 -> Resistor_SMD:R_1206_3216Metric_Pad1.30x1.75mm_HandSolder
- R74: footprint Resistor-1206-Footprints:R74 -> Resistor_SMD:R_1206_3216Metric_Pad1.30x1.75mm_HandSolder
- R75, R751: footprint Resistor-1206-Footprints:R75 -> Resistor_SMD:R_1206_3216Metric_Pad1.30x1.75mm_HandSolder
- R76, R762: footprint Resistor-1206-Footprints:R76 -> Resistor_SMD:R_1206_3216Metric_Pad1.30x1.75mm_HandSolder
- R77, R90: footprint Resistor-1206-Footprints:R77 -> Resistor_SMD:R_1206_3216Metric_Pad1.30x1.75mm_HandSolder
- R8: footprint Resistor-1206-Footprints:R8 -> Resistor_SMD:R_1206_3216Metric_Pad1.30x1.75mm_HandSolder
- R89: footprint Resistor-1206-Footprints:R89 -> Resistor_SMD:R_1206_3216Metric_Pad1.30x1.75mm_HandSolder
- moved C19 343.7 mm to (197.5, 114.6), turned to 90 degrees
- moved C18 335.6 mm to (195.0, 71.9), turned to 90 degrees
- moved C98 328.6 mm to (195.0, 85.9), turned to -90 degrees
- moved R7 324.0 mm to (228.9, 70.0)
- moved R72 322.2 mm to (237.5, 71.0)
- moved C23 316.9 mm to (220.5, 68.5), turned to 90 degrees
- moved C89 315.2 mm to (221.0, 90.0), turned to -90 degrees
- moved R78 314.7 mm to (236.6, 37.6)
- moved R79 314.6 mm to (236.6, 40.1)
- moved C22 313.9 mm to (217.0, 68.5), turned to 90 degrees
- moved C26 312.7 mm to (217.5, 90.0), turned to -90 degrees
- moved C21 311.0 mm to (213.5, 68.5), turned to 90 degrees
- moved R751 310.2 mm to (220.5, 105.0)
- moved C25 310.2 mm to (214.0, 90.0), turned to -90 degrees
- moved C24 309.2 mm to (210.5, 89.9), turned to -90 degrees
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Connections:
- C27 pad 2: +BATT -> V_BAT+
- C28 pad 2: +BATT -> V_BAT+
- C29 pad 2: +BATT -> V_BAT+
- C30 pad 2: +BATT -> V_BAT+
- C508 pad 2: 12V -> Net-(C508-C2)
- C94 pad 2: +BATT -> V_BAT+
- L1 pad 2: 12V -> Net-(C508-C2)
- Q1 pad 10: +BATT -> V_BAT+
- Q1 pad 11: +BATT -> V_BAT+
- Q1 pad 12: +BATT -> V_BAT+
- Q1 pad 13: +BATT -> V_BAT+
- Q1 pad 14: +BATT -> V_BAT+
- Q1 pad 15: +BATT -> V_BAT+
- Q1 pad 16: +BATT -> V_BAT+
- Q1 pad 9: +BATT -> V_BAT+
- R10 pad 1: +BATT -> V_BAT+
- R502 pad 1: 12V -> Net-(C508-C2)
Routing:
- net V_BAT-: vias 0 -> 14
- net V_BAT+: vias 0 -> 26
- net 5V: vias 0 -> 7
- net /U-Phase/U_CS+: vias 0 -> 11
- net /U-Phase/U: vias 0 -> 37
- added copper zone on In2.Cu, net 5V
- removed copper zone on In2.Cu, net /U-Phase/+5V
- removed copper zone on In2.Cu, net /U-Phase/12V
- removed copper zone on In2.Cu, net 12V
- removed copper zone on In3.Cu, net 5V
- removed copper zone on In1.Cu, net GND
- removed copper zone on In4.Cu, net GNDS

Commit message: v07112024
Parts:
- added G***: LOGO, 1206-Infineon-Library:Aryan-Pepe-Logo, F.Cu at (227.0, 129.5)
- moved R74 330.3 mm to (236.0, 109.5), turned to 180 degrees
- moved C80 306.9 mm to (236.0, 112.0)
- moved R73 301.2 mm to (236.1, 114.5), turned to 180 degrees
- moved C77 252.6 mm to (206.5, 38.5), turned to 180 degrees
- moved C35 239.4 mm to (144.5, 96.0), turned to 90 degrees
- moved R81 232.9 mm to (138.5, 123.0)
- moved D4 37.7 mm to (146.6, 106.3), turned to 90 degrees
- moved R12 32.1 mm to (150.0, 108.0), turned to 0 degrees
- moved R11 30.4 mm to (150.0, 104.7), turned to 0 degrees
- moved R13 29.9 mm to (150.1, 102.3), turned to 0 degrees
- moved C94 29.1 mm to (150.5, 65.0), turned to 180 degrees
- moved R63 14.8 mm to (189.0, 43.5)
- moved C72 13.7 mm to (113.0, 46.5)
- moved POT1 13.7 mm to (106.5, 48.0)
- moved R61 13.7 mm to (104.0, 42.5)
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Routing:
- net V_BAT-: track 0.00 -> 111.4 mm, vias 14 -> 22
- net V_BAT+: track 0.00 -> 94.0 mm, vias 26 -> 27
- net /U-Phase/U: track 0.00 -> 45.7 mm
- net /Power Board Connector/DR_EN: track 0.00 -> 42.0 mm, vias 0 -> 2
- net GND: track 0.00 -> 39.8 mm, vias 0 -> 9
- net +5V: track 0.00 -> 24.8 mm, vias 0 -> 9
- net Net-(IC1-SW): track 0.00 -> 23.1 mm, vias 0 -> 2
- net /U-Phase/U_CS+: track 0.00 -> 22.1 mm
- net Net-(D12-K): track 0.00 -> 21.0 mm, vias 0 -> 2
- net GNDS: track 0.00 -> 16.9 mm, vias 0 -> 4
- net Net-(OP5--IN): track 0.00 -> 16.3 mm
- net 12V: track 0.00 -> 16.0 mm
- net Net-(OP1--IN): track 0.00 -> 14.3 mm, vias 0 -> 2
- net Net-(OP1-OUT): track 0.00 -> 13.1 mm
- net Net-(IC1-FB): track 0.00 -> 12.6 mm
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- added copper zone on In3.Cu, net +5V
- added copper zone on In1.Cu, net GND
- added copper zone on In1.Cu, net GNDS
- added copper zone on In4.Cu, net OFFSET
- removed copper zone on In2.Cu, net 5V

Commit message: v07112024
Parts:
- removed G***: LOGO, 1206-Infineon-Library:Aryan-Pepe-Logo
- J3: footprint infineon-library-footprints:TSW-103-08-L-S -> just-footprints:SAMTEC_TSW-103-08-L-S
- moved R762 47.1 mm to (179.4, 95.0)
- moved RT2 40.7 mm to (179.9, 98.0), turned to 90 degrees
- moved R751 37.8 mm to (183.4, 97.5), turned to 90 degrees
- moved C811 36.6 mm to (178.4, 102.5), turned to 90 degrees
- moved C821 34.3 mm to (180.9, 102.5), turned to 90 degrees
- moved R16 12.0 mm to (150.5, 75.0)
- moved C84 10.7 mm to (137.0, 116.6), turned to -90 degrees
- moved D5 9.47 mm to (146.5, 76.5), turned to 90 degrees
- moved R82 9.22 mm to (139.5, 116.5), turned to -90 degrees
- moved C83 8.01 mm to (143.7, 115.0), turned to 0 degrees
- moved R81 7.45 mm to (143.5, 117.5)
- moved R12 7.00 mm to (150.1, 101.0)
- moved R18 7.00 mm to (150.5, 77.5)
- moved C37 4.95 mm to (143.0, 122.5), turned to 180 degrees
- moved R13 3.76 mm to (150.5, 106.0)
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- renumbered REF** to M1, REF** to M2, REF** to M3, REF** to M4
Connections:
- net +BATT renamed V_BATT+
Routing:
- net V_BAT-: track 111.4 -> 171.9 mm
- net 5V: track 5.50 -> 37.7 mm, vias 0 -> 4
- net /U-Phase/U-LI: track 0.00 -> 32.1 mm, vias 0 -> 2
- net /U-Phase/U-HI: track 0.00 -> 31.9 mm, vias 0 -> 2
- net Net-(D5-A): track 0.00 -> 27.6 mm, vias 0 -> 2
- net Net-(D4-A): track 0.00 -> 21.4 mm
- net /U-Phase/U-LO: track 0.00 -> 20.6 mm
- net Net-(U13-CLK): track 12.0 -> 32.1 mm
- net GND: track 39.8 -> 54.3 mm, vias 9 -> 16
- net Net-(Q8-G): track 9.62 -> 23.9 mm
- net Net-(D15-K): track 7.99 -> 22.1 mm, vias 0 -> 1
- net Net-(OP5-+IN): track 8.27 -> 19.6 mm, vias 0 -> 2
- net SD: track 6.36 -> 17.5 mm
- net /U-Phase/U-HIN: track 0.00 -> 11.1 mm, vias 0 -> 2
- net +5V: track 24.8 -> 34.9 mm, vias 9 -> 10
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
Commit message: v08112024
Parts:
- added G***: LOGO, 1206-Infineon-Library:Aryan-Pepe-Logo, F.Cu at (227.5, 132.5)
- J3: footprint just-footprints:SAMTEC_TSW-103-08-L-S -> just-footprints:SAMTEC_HTSW-103-XX-X-S
- L1: footprint Misc-Footprints:L1 -> Inductor_SMD:L_1206_3216Metric
- moved R75 20.0 mm to (187.5, 71.0)
- moved R78 11.2 mm to (236.5, 45.5), turned to 90 degrees
- moved J4 7.81 mm to (107.0, 135.0)
- moved R73 7.50 mm to (236.0, 107.0)
- moved R503 6.53 mm to (106.0, 124.5)
- moved C508 6.52 mm to (111.2, 127.0)
- moved R501 6.52 mm to (106.1, 127.0)
- moved R502 6.52 mm to (111.2, 124.5)
- moved C506 5.59 mm to (99.5, 130.0)
- moved C507 5.59 mm to (99.8, 119.6)
- moved IC1 5.59 mm to (100.4, 124.8)
- moved D15 4.50 mm to (240.0, 107.7)
- moved L1 4.22 mm to (112.7, 121.0), turned to -90 degrees
- moved RT1 2.67 mm to (180.5, 83.5), turned to 90 degrees
- moved C81 2.25 mm to (183.5, 77.0)
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Connections:
- C62 pad 2: Net-(OP1-OUT) -> I_PHASE_U
- OP1 pad 1: Net-(OP1-OUT) -> I_PHASE_U
- R46 pad 2: Net-(OP1-OUT) -> I_PHASE_U
- R47 pad 1: Net-(OP1-OUT) -> I_PHASE_U
- R73 pad 2: V_BATT+ -> V_BAT+
Routing:
- net V_BAT-: track 171.9 -> 394.3 mm, vias 22 -> 7
- net V_BAT+: track 97.0 -> 311.0 mm, vias 27 -> 7
- net SD: track 17.5 -> 217.8 mm, vias 0 -> 1
- net I_SNS_PHASE_U: track 4.70 -> 205.0 mm
- net U-L: track 0.18 -> 147.7 mm, vias 0 -> 5
- net BEMF_PHASE_U: track 2.52 -> 122.1 mm, vias 0 -> 2
- net I_PHASE_U: track 0.00 -> 104.5 mm, vias 0 -> 4
- net OFFSET: track 9.29 -> 112.1 mm, vias 3 -> 5
- net Net-(C811-Pad2): track 0.00 -> 90.4 mm, vias 0 -> 5
- net Net-(C81-Pad2): track 0.00 -> 72.2 mm
- net GNDS: track 25.0 -> 76.7 mm, vias 5 -> 8
- net /U-Phase/U_CS+: track 21.8 -> 55.4 mm, vias 10 -> 5
- net /Power Board Connector/DR_EN: track 44.9 -> 76.3 mm, vias 2 -> 1
- net GND: track 54.3 -> 80.1 mm, vias 16 -> 22
- net /U-Phase/U: track 37.9 -> 61.7 mm, vias 37 -> 8
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- added copper zone on In4.Cu, net GNDS
- removed copper zone on In1.Cu, net GNDS
- removed copper zone on In4.Cu, net OFFSET
