File: EVAL-TOLT-DC48V-3KW-TOBO2-1206/EVAL_TOLT_DC48V_3KW.kicad_pcb (KiCad board)
At the start: 6 copper layers, 170 x 120 mm, 149 parts, among them IC1 LM5013QDDARQ1, J1 V_BAT+, J12 Direction Switch, J2 V_BAT-, J3 EXT/ITN 12V, J4 +12V_EXT, J5 +5V_EXT, M1 MountingHole_3.2mm_M3_DIN965, M2 MountingHole_3.2mm_M3_DIN965, M3 MountingHole_3.2mm_M3_DIN965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

Commit message: v08112024
Added Heatsink Mounting Holes
Parts:
- added K1: MountingHole_3.2mm_M3_DIN965, MountingHole:MountingHole_3.2mm_M3_DIN965, F.Cu at (145.5, 119.5)
- added K2: MountingHole_3.2mm_M3_DIN965, MountingHole:MountingHole_3.2mm_M3_DIN965, F.Cu at (184.0, 51.5)
- moved C83 8.74 mm to (136.3, 119.7)
- moved U4 8.74 mm to (135.7, 124.7)
- moved C37 8.74 mm to (135.6, 127.2)
- moved C84 8.74 mm to (129.6, 121.3)
- moved R81 8.74 mm to (136.1, 122.2)
- moved R82 8.74 mm to (132.1, 121.2)
- moved C78 6.21 mm to (188.0, 55.0)
- moved R71 2.07 mm to (190.5, 52.5), turned to 90 degrees
- renumbered G*** to LOGO
Routing:
- net /U-Phase/U-LI: track 33.3 -> 42.6 mm
- net SD: track 217.8 -> 227.2 mm
- net U-L: track 147.7 -> 156.6 mm
- net /U-Phase/U-HI: track 31.5 -> 40.3 mm
- net GND: track 80.1 -> 82.6 mm
- net +5V: track 49.6 -> 50.5 mm

Commit message: v10112024
Parts:
- added C505: 12061C225KAT2A, Capacitor_SMD:C_1206_3216Metric, F.Cu at (99.5, 132.5)
- added C509: 12061C273KAT2A, Capacitor_SMD:C_1206_3216Metric, F.Cu at (110.0, 121.0)
- added C510: 47 pF, 115 mOhm, Capacitor_SMD:C_1206_3216Metric_Pad1.33x1.80mm_HandSolder, F.Cu at (109.5, 115.0)
- added C511: 3.3 nF, 332 mOhm, Capacitor_SMD:C_1206_3216Metric_Pad1.33x1.80mm_HandSolder, F.Cu at (115.5, 121.1)
- added D1: 770 mV, 5.5 A, Diode_SMD:D_1206_3216Metric, F.Cu at (96.0, 124.0)
- added R504: 221 kOhm, Resistor_SMD:R_1206_3216Metric_Pad1.30x1.75mm_HandSolder, F.Cu at (115.5, 116.1)
- D12: footprint Misc-Footprints:D12 -> Diode_SMD:D_1206_3216Metric_Pad1.42x1.75mm_HandSolder
- D15: footprint Misc-Footprints:D15 -> Diode_SMD:D_1206_3216Metric_Pad1.42x1.75mm_HandSolder
- D3: footprint Misc-Footprints:D3 -> Diode_SMD:D_1206_3216Metric_Pad1.42x1.75mm_HandSolder
- D4, D5: footprint Misc-Footprints:D4 -> Diode_SMD:D_1206_3216Metric_Pad1.42x1.75mm_HandSolder
- J3: footprint just-footprints:SAMTEC_HTSW-103-XX-X-S -> Connector_PinHeader_2.54mm:PinHeader_1x03_P2.54mm_Vertical
- J4: footprint Misc-Footprints:J4 -> Connector_PinHeader_2.54mm:PinHeader_1x02_P2.54mm_Vertical
- L1: footprint Inductor_SMD:L_1206_3216Metric -> Inductor_SMD:L_1206_3216Metric_Pad1.22x1.90mm_HandSolder
- U12: footprint Misc-Footprints:PCN -> Connector_IDC:IDC-Header_2x17_P2.54mm_Vertical
- moved U12 39.4 mm to (243.7, 69.6), turned to 0 degrees
- moved C80 5.69 mm to (230.4, 113.3)
- moved D15 5.69 mm to (234.5, 109.0)
- moved R73 5.69 mm to (230.5, 108.3)
- moved R74 5.69 mm to (230.4, 110.8)
- moved D4 1.75 mm to (146.2, 104.2)
- moved J3 0.86 mm to (116.0, 128.9), turned to 0 degrees
- moved L1 0.28 mm to (112.7, 120.7)
- moved J4 0.12 mm to (106.9, 134.9)
- moved OP1 0.08 mm to (135.3, 50.7)
Connections:
- C16 pad 2: 5V -> +5V
- C17 pad 2: 5V -> +5V
- C32 pad 1: /U-Phase/U_CS+ -> U_CS+
- C94 pad 1: /U-Phase/U_CS+ -> U_CS+
- G1 pad 2: 5V -> +5V
- J5 pad 2: 5V -> +5V
- Q4 pad 1: /U-Phase/U_CS+ -> U_CS+
- Q4 pad 2: /U-Phase/U_CS+ -> U_CS+
- Q4 pad 3: /U-Phase/U_CS+ -> U_CS+
- Q4 pad 4: /U-Phase/U_CS+ -> U_CS+
- Q4 pad 5: /U-Phase/U_CS+ -> U_CS+
- Q4 pad 6: /U-Phase/U_CS+ -> U_CS+
- Q4 pad 7: /U-Phase/U_CS+ -> U_CS+
- R1 pad 2: 5V -> +5V
- R19 pad 2: /U-Phase/U_CS+ -> U_CS+
- R8 pad 1: 5V -> +5V
- RS1 pad 1: /U-Phase/U_CS+ -> U_CS+
- TP2 pad 1: 5V -> +5V
- U3 pad 7: /U-Phase/U_CS+ -> U_CS+
- U3 pad 9: /U-Phase/U_CS+ -> U_CS+
Routing:
- net U_CS+: track 0.00 -> 92.9 mm, vias 0 -> 14
- net /U-Phase/U: track 61.7 -> 124.3 mm, vias 8 -> 50
- net /U-Phase/U_CS+: track 55.4 -> 0.00 mm, vias 5 -> 0
- net U-L: track 156.6 -> 208.9 mm, vias 5 -> 1
- net 5V: track 41.3 -> 0.00 mm, vias 3 -> 0
- net SD: track 227.2 -> 267.4 mm, vias 1 -> 2
- net GNDS: track 76.7 -> 37.7 mm, vias 8 -> 9
- net +5V: track 50.5 -> 73.4 mm, vias 13 -> 19
- net GND: track 82.6 -> 62.0 mm, vias 22 -> 24
- net Net-(C81-Pad2): track 72.2 -> 91.9 mm
- net 12V: track 32.4 -> 14.0 mm
- net I_PHASE_U: track 104.5 -> 87.7 mm, vias 4 -> 2
- net I_SNS_PHASE_U: track 205.0 -> 188.3 mm, vias 1 -> 3
- net V_BAT-: track 394.3 -> 407.4 mm, vias 7 -> 24
- net BEMF_PHASE_U: track 122.1 -> 109.3 mm
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- added copper zone on In1.Cu, net /U-Phase/U
- added copper zone on In3.Cu, net /U-Phase/U
- added copper zone on In4.Cu, net /U-Phase/U
- added copper zone on In2.Cu, net 12V
- added copper zone on In1.Cu, net U_CS+
- added copper zone on In2.Cu, net U_CS+
- added copper zone on In3.Cu, net U_CS+
- added copper zone on In4.Cu, net U_CS+
- added copper zone on In1.Cu, net V_BAT+
- added copper zone on In3.Cu, net V_BAT+
- added copper zone on In4.Cu, net V_BAT+
- added copper zone on In1.Cu, net V_BAT-
- added copper zone on In3.Cu, net V_BAT-
- added copper zone on In4.Cu, net V_BAT-
- removed copper zone on In2.Cu, net /U-Phase/U_CS+

Commit message: v10112024-2
Parts:
- C510, C511: footprint Capacitor_SMD:C_1206_3216Metric_Pad1.33x1.80mm_HandSolder -> Capacitor_SMD:C_1206_3216Metric
- J12: footprint Misc-Footprints:J12 -> Connector_PinHeader_2.54mm:PinHeader_1x02_P2.54mm_Vertical
- moved R75 17.4 mm to (179.8, 86.6), turned to 180 degrees
- moved C82 10.4 mm to (181.7, 88.9), turned to 0 degrees
- moved R76 3.85 mm to (184.6, 83.2)
- moved C81 3.57 mm to (181.8, 80.2)
- moved RT1 0.38 mm to (180.1, 83.4)
- moved J3 0.35 mm to (115.8, 129.2)
- turned J12 to 0 degrees
Connections:
- C82 pad 1: Net-(RT1-GND) -> GNDS
- C82 pad 2: GNDS -> Net-(RT1-V_{DD})
- J12 pad 1: (no net) -> GNDS
- J12 pad 2: (no net) -> Net-(J12-Pad2)
- J3 pad 1: (no net) -> Net-(C508-C2)
- J3 pad 2: (no net) -> 12V
- J3 pad 3: (no net) -> Net-(J3-Pad3)
- J4 pad 2: Net-(J3-Pad03) -> Net-(J3-Pad3)
- R72 pad 1: Net-(J12-Pad02) -> Net-(J12-Pad2)
- R75 pad 1: GNDS -> Net-(RT1-V_{DD})
- RT1 pad 1: GNDS -> Net-(RT1-V_{DD})
- RT1 pad 3: Net-(RT1-GND) -> GNDS
Routing:
- net GNDS: track 37.7 -> 50.6 mm, vias 9 -> 7
- net OFFSET: track 108.0 -> 95.9 mm, vias 3 -> 2
- net Net-(J3-Pad3): track 0.00 -> 10.2 mm
- net Net-(RT1-V_{DD}): track 0.00 -> 5.40 mm
- net Net-(J12-Pad2): track 0.00 -> 4.60 mm
- net 12V: track 14.0 -> 18.1 mm
- net Net-(C508-C2): track 10.7 -> 14.7 mm
- net Net-(RT1-GND): track 3.49 -> 0.00 mm
- net /U-Phase/U: track 124.3 -> 121.2 mm
- net Net-(C81-Pad2): track 91.9 -> 93.9 mm
- net Net-(D15-K): track 30.2 -> 28.8 mm, vias 1 -> 0
- net Net-(RT1-V_{OUT}): track 3.30 -> 2.25 mm
- net Net-(IC1-FB): vias 1 -> 0
