File: EVAL-TOLT-DC48V-3KW-TOBO2-1206/EVAL_TOLT_DC48V_3KW.kicad_pcb (KiCad board)
At the start: 6 copper layers, 170 x 120 mm, 157 parts, among them IC1 LM5013QDDARQ1, J1 V_BAT+, J12 Direction Switch, J2 V_BAT-, J3 EXT/ITN 12V, J4 +12V_EXT, J5 +5V_EXT, K1 MountingHole_3.2mm_M3_DIN965, K2 MountingHole_3.2mm_M3_DIN965, M1 MountingHole_3.2mm_M3_DIN965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

Commit message: v11112024
Parts:
- moved K1 1.58 mm to (145.0, 121.0)
- moved K2 1.58 mm to (183.5, 53.0)

Commit message: v11112024-2
Parts:
- moved C821 1.85 mm to (182.0, 104.0), turned to 0 degrees
- moved Q7 0.45 mm to (231.0, 44.5)
Routing:
- net Net-(RT2-V_{DD}): track 9.45 -> 7.49 mm
- net GNDS: track 50.6 -> 51.2 mm
