File: EVAL-TOLT-DC48V-3KW-TOBO2-1206/Current Offset.kicad_sch (KiCad schematic)
At the start: 8 parts

Commit message: v06112024
Parts:
- C72: footprint Kap-1206-Footprints:C72 -> Capacitor_SMD:C_1206_3216Metric
- C73: footprint Kap-1206-Footprints:C15 -> Capacitor_SMD:C_1206_3216Metric
- R60: footprint Resistor-1206-Footprints:R60 -> Resistor_SMD:R_1206_3216Metric_Pad1.30x1.75mm_HandSolder
- R61: footprint Resistor-1206-Footprints:R61 -> Resistor_SMD:R_1206_3216Metric_Pad1.30x1.75mm_HandSolder
- R62: footprint Resistor-1206-Footprints:R12 -> Resistor_SMD:R_1206_3216Metric_Pad1.30x1.75mm_HandSolder
Changed lines of the file:
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@@
 			)
 		)
-		(property "Footprint" "Resistor-1206-Footprints:R60"
+		(property "Footprint" "Resistor_SMD:R_1206_3216Metric_Pad1.30x1.75mm_HandSolder"
 			(at 77.47 32.512 90)
 			(effects
@@
 			)
 		)
-		(property "Footprint" "Resistor-1206-Footprints:R61"
+		(property "Footprint" "Resistor_SMD:R_1206_3216Metric_Pad1.30x1.75mm_HandSolder"
 			(at 78.74 95.758 90)
 			(effects
@@
 			)
 		)
-		(property "Footprint" "Kap-1206-Footprints:C15"
+		(property "Footprint" "Capacitor_SMD:C_1206_3216Metric"
 			(at 147.32 56.1848 0)
 			(effects
@@
 			)
 		)
-		(property "Footprint" "Kap-1206-Footprints:C72"
+		(property "Footprint" "Capacitor_SMD:C_1206_3216Metric"
 			(at 50.8 82.8548 0)
 			(effects
@@
 			)
 		)
-		(property "Footprint" "Resistor-1206-Footprints:R12"
+		(property "Footprint" "Resistor_SMD:R_1206_3216Metric_Pad1.30x1.75mm_HandSolder"
 			(at 143.51 33.528 90)
 			(effects

Commit message: v11112024-3
Parts:
- TP3: footprint TestPoint:TestPoint_Bridge_Pitch2.54mm_Drill0.7mm -> TestPoint:TestPoint_Pad_3.0x3.0mm
Changed lines of the file:
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@@
 			)
 		)
-		(property "Footprint" "TestPoint:TestPoint_Bridge_Pitch2.54mm_Drill0.7mm"
+		(property "Footprint" "TestPoint:TestPoint_Pad_3.0x3.0mm"
 			(at 184.785 68.58 0)
 			(effects
