File: EVAL-TOLT-DC48V-3KW-TOBO2-1206/Current Comparator & Latch.kicad_sch (KiCad schematic)
At the start: 29 parts, among them Q8 IRLML6346, U11 LMV331, U13 SN74LVC2G74DCUR

Commit message: v06112024
Parts:
- C74, C93: footprint Kap-1206-Footprints:C72 -> Capacitor_SMD:C_1206_3216Metric
- C75, C78, C92: footprint Kap-1206-Footprints:C15 -> Capacitor_SMD:C_1206_3216Metric
- C76: footprint Kap-1206-Footprints:C76 -> Capacitor_SMD:C_1206_3216Metric
- C77, C79: footprint Kap-1206-Footprints:C8 -> Capacitor_SMD:C_1206_3216Metric
- R63: footprint Resistor-1206-Footprints:R63 -> Resistor_SMD:R_1206_3216Metric_Pad1.30x1.75mm_HandSolder
- R64: footprint Resistor-1206-Footprints:R64 -> Resistor_SMD:R_1206_3216Metric_Pad1.30x1.75mm_HandSolder
- R67, R68, R71: footprint Resistor-1206-Footprints:R61 -> Resistor_SMD:R_1206_3216Metric_Pad1.30x1.75mm_HandSolder
- R69: footprint Resistor-1206-Footprints:R12 -> Resistor_SMD:R_1206_3216Metric_Pad1.30x1.75mm_HandSolder
- R70: footprint Resistor-1206-Footprints:R70 -> Resistor_SMD:R_1206_3216Metric_Pad1.30x1.75mm_HandSolder
- R87, R88: footprint Resistor-1206-Footprints:R72 -> Resistor_SMD:R_1206_3216Metric_Pad1.30x1.75mm_HandSolder
- R89: footprint Resistor-1206-Footprints:R89 -> Resistor_SMD:R_1206_3216Metric_Pad1.30x1.75mm_HandSolder
- R90: footprint Resistor-1206-Footprints:R77 -> Resistor_SMD:R_1206_3216Metric_Pad1.30x1.75mm_HandSolder
Changed lines of the file:
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@@
 	)
 	(junction
-		(at 45.72 153.035)
-		(diameter 0)
-		(color 0 0 0 0)
-	)
-	(junction
 		(at 166.37 63.5)
 		(diameter 0)
@@
 	)
 	(junction
+		(at 45.72 153.67)
+		(diameter 0)
+		(color 0 0 0 0)
+	)
+	(junction
 		(at 137.16 60.96)
 		(diameter 0)
@@
 	(wire
 		(pts
-			(xy 45.72 143.51) (xy 45.72 153.035)
-		)
-		(stroke
-			(width 0)
-			(type default)
-		)
-	)
-	(wire
-		(pts
 			(xy 104.14 60.96) (xy 137.16 60.96)
 		)
@@
 	(wire
 		(pts
-			(xy 22.225 151.765) (xy 22.86 151.765)
+			(xy 124.46 80.01) (xy 124.46 66.04)
 		)
 		(stroke
@@
 	(wire
 		(pts
-			(xy 124.46 80.01) (xy 124.46 66.04)
+			(xy 241.3 66.04) (xy 241.3 57.785)
 		)
 		(stroke
@@
 	(wire
 		(pts
-			(xy 241.3 66.04) (xy 241.3 57.785)
+			(xy 150.495 71.12) (xy 150.495 74.93)
 		)
 		(stroke
@@
 	(wire
 		(pts
-			(xy 150.495 71.12) (xy 150.495 74.93)
+			(xy 88.646 105.41) (xy 98.425 105.41)
 		)
 		(stroke
@@
 	(wire
 		(pts
-			(xy 88.646 105.41) (xy 98.425 105.41)
+			(xy 71.12 38.1) (xy 71.12 30.48)
 		)
 		(stroke
@@
 	(wire
 		(pts
-			(xy 71.12 38.1) (xy 71.12 30.48)
+			(xy 45.72 143.51) (xy 45.72 153.67)
 		)
 		(stroke
@@
 	(wire
 		(pts
-			(xy 22.86 151.765) (xy 22.86 127)
+			(xy 22.86 127) (xy 22.86 153.67)
 		)
 		(stroke
@@
 	(wire
 		(pts
-			(xy 22.225 151.765) (xy 22.225 153.035)
-		)
-		(stroke
-			(width 0)
-			(type default)
-		)
-	)
-	(wire
-		(pts
 			(xy 42.545 116.205) (xy 38.1 116.205)
 		)
@@
 	(wire
 		(pts
-			(xy 22.225 153.035) (xy 45.72 153.035)
+			(xy 22.86 153.67) (xy 45.72 153.67)
 		)
 		(stroke
@@
 	(wire
 		(pts
-			(xy 45.72 153.035) (xy 45.72 153.67)
-		)
-		(stroke
-			(width 0)
-			(type default)
-		)
-	)
-	(wire
-		(pts
 			(xy 33.02 30.48) (xy 38.1 30.48)
 		)
@@
 			)
 		)
-		(property "Footprint" "Kap-1206-Footprints:C15"
+		(property "Footprint" "Capacitor_SMD:C_1206_3216Metric"
 			(at 91.44 87.9348 0)
 			(effects
@@
 			)
 		)
-		(property "Footprint" "Resistor-1206-Footprints:R61"
+		(property "Footprint" "Resistor_SMD:R_1206_3216Metric_Pad1.30x1.75mm_HandSolder"
 			(at 45.72 102.108 90)
 			(effects
@@
 			)
 		)
-		(property "Footprint" "Kap-1206-Footprints:C15"
+		(property "Footprint" "Capacitor_SMD:C_1206_3216Metric"
 			(at 138.43 42.2148 0)
 			(effects
@@
 			)
 		)
-		(property "Footprint" "Resistor-1206-Footprints:R63"
+		(property "Footprint" "Resistor_SMD:R_1206_3216Metric_Pad1.30x1.75mm_HandSolder"
 			(at 46.482 30.48 90)
 			(effects
@@
 			)
 		)
-		(property "Footprint" "Kap-1206-Footprints:C8"
+		(property "Footprint" "Capacitor_SMD:C_1206_3216Metric"
 			(at 128.27 86.6648 0)
 			(effects
@@
 			)
 		)
-		(property "Footprint" "Kap-1206-Footprints:C72"
+		(property "Footprint" "Capacitor_SMD:C_1206_3216Metric"
 			(at 26.67 126.0348 0)
 			(effects
@@
 			)
 		)
-		(property "Footprint" "Kap-1206-Footprints:C8"
+		(property "Footprint" "Capacitor_SMD:C_1206_3216Metric"
 			(at 187.96 77.7748 0)
 			(effects
@@
 			)
 		)
-		(property "Footprint" "Kap-1206-Footprints:C76"
+		(property "Footprint" "Capacitor_SMD:C_1206_3216Metric"
 			(at 107.95 70.1548 0)
 			(effects
@@
 			)
 		)
-		(property "Footprint" "Resistor-1206-Footprints:R77"
+		(property "Footprint" "Resistor_SMD:R_1206_3216Metric_Pad1.30x1.75mm_HandSolder"
 			(at 241.3 64.262 90)
 			(effects
@@
 			)
 		)
-		(property "Footprint" "Resistor-1206-Footprints:R89"
+		(property "Footprint" "Resistor_SMD:R_1206_3216Metric_Pad1.30x1.75mm_HandSolder"
 			(at 203.2 86.868 90)
 			(effects
@@
 			)
 		)
-		(property "Footprint" "Resistor-1206-Footprints:R70"
+		(property "Footprint" "Resistor_SMD:R_1206_3216Metric_Pad1.30x1.75mm_HandSolder"
 			(at 144.272 87.63 90)
 			(effects
@@
 			)
 		)
-		(property "Footprint" "Resistor-1206-Footprints:R72"
+		(property "Footprint" "Resistor_SMD:R_1206_3216Metric_Pad1.30x1.75mm_HandSolder"
 			(at 254 83.058 90)
 			(effects
@@
 			)
 		)
-		(property "Footprint" "Resistor-1206-Footprints:R64"
+		(property "Footprint" "Resistor_SMD:R_1206_3216Metric_Pad1.30x1.75mm_HandSolder"
 			(at 28.702 38.1 90)
 			(effects
@@
 			)
 		)
-		(property "Footprint" "Resistor-1206-Footprints:R12"
+		(property "Footprint" "Resistor_SMD:R_1206_3216Metric_Pad1.30x1.75mm_HandSolder"
 			(at 87.63 65.278 90)
 			(effects
@@
 			)
 		)
-		(property "Footprint" "Kap-1206-Footprints:C15"
+		(property "Footprint" "Capacitor_SMD:C_1206_3216Metric"
 			(at 209.55 42.2148 0)
 			(effects
@@
 			)
 		)
-		(property "Footprint" "Resistor-1206-Footprints:R61"
+		(property "Footprint" "Resistor_SMD:R_1206_3216Metric_Pad1.30x1.75mm_HandSolder"
 			(at 166.37 40.132 90)
 			(effects
@@
 			)
 		)
-		(property "Footprint" "Resistor-1206-Footprints:R61"
+		(property "Footprint" "Resistor_SMD:R_1206_3216Metric_Pad1.30x1.75mm_HandSolder"
 			(at 45.72 145.288 90)
 			(effects
@@
 			)
 		)
-		(property "Footprint" "Resistor-1206-Footprints:R72"
+		(property "Footprint" "Resistor_SMD:R_1206_3216Metric_Pad1.30x1.75mm_HandSolder"
 			(at 264.16 42.418 90)
 			(effects
@@
 			)
 		)
-		(property "Footprint" "Kap-1206-Footprints:C72"
+		(property "Footprint" "Capacitor_SMD:C_1206_3216Metric"
 			(at 207.01 104.4448 0)
 			(effects

Commit message: v10112024
Parts:
- D12: footprint Misc-Footprints:D12 -> Diode_SMD:D_1206_3216Metric_Pad1.42x1.75mm_HandSolder
Changed lines of the file:
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@@
 			)
 		)
-		(property "Footprint" "Misc-Footprints:D12"
+		(property "Footprint" "Diode_SMD:D_1206_3216Metric_Pad1.42x1.75mm_HandSolder"
 			(at 59.69 38.1 0)
 			(effects

Commit message: v11112024-3
Parts:
- TP4, TP5, TP6: footprint TestPoint:TestPoint_Bridge_Pitch2.54mm_Drill0.7mm -> TestPoint:TestPoint_Pad_3.0x3.0mm
Changed lines of the file:
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@@
 			)
 		)
-		(property "Footprint" "TestPoint:TestPoint_Bridge_Pitch2.54mm_Drill0.7mm"
+		(property "Footprint" "TestPoint:TestPoint_Pad_3.0x3.0mm"
 			(at 190.5 53.34 0)
 			(effects
@@
 			)
 		)
-		(property "Footprint" "TestPoint:TestPoint_Bridge_Pitch2.54mm_Drill0.7mm"
+		(property "Footprint" "TestPoint:TestPoint_Pad_3.0x3.0mm"
 			(at 278.765 30.48 0)
 			(effects
@@
 			)
 		)
-		(property "Footprint" "TestPoint:TestPoint_Bridge_Pitch2.54mm_Drill0.7mm"
+		(property "Footprint" "TestPoint:TestPoint_Pad_3.0x3.0mm"
 			(at 107.95 100.33 0)
 			(effects

Commit message: v15112024
Parts:
- D12: footprint Diode_SMD:D_1206_3216Metric_Pad1.42x1.75mm_HandSolder -> Diode_SMD:D_SOD-323F
Changed lines of the file:
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@@
 			)
 		)
-		(property "Footprint" "Diode_SMD:D_1206_3216Metric_Pad1.42x1.75mm_HandSolder"
+		(property "Footprint" "Diode_SMD:D_SOD-323F"
 			(at 59.69 38.1 0)
 			(effects
