File: EVAL-TOLT-DC48V-3KW-TOBO2-1206/Current amplifier.kicad_sch (KiCad schematic)
At the start: 27 parts, among them J1 V_BAT+, J2 V_BAT-

Commit message: v01112024
New PCB Version for Zones
Connections:
- net V_BAT+: now reaches C18.2, C19.2, C20.2, C21.2, C22.2, C23.2, C24.2, C25.2, C26.2, C89.2, C97.2, C98.2, C99.2, J1.1 (Pin_1)
Changed lines of the file:
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@@
 	)
 	(junction
+		(at 46.99 133.35)
+		(diameter 0)
+		(color 0 0 0 0)
+	)
+	(junction
 		(at 196.85 106.68)
 		(diameter 0)
@@
 	)
 	(junction
+		(at 48.26 106.68)
+		(diameter 0)
+		(color 0 0 0 0)
+	)
+	(junction
 		(at 120.65 133.35)
 		(diameter 0)
@@
 	(wire
 		(pts
+			(xy 46.99 135.89) (xy 46.99 133.35)
+		)
+		(stroke
+			(width 0)
+			(type default)
+		)
+	)
+	(wire
+		(pts
 			(xy 95.25 106.68) (xy 107.95 106.68)
 		)
@@
 	(wire
 		(pts
+			(xy 48.26 104.14) (xy 48.26 106.68)
+		)
+		(stroke
+			(width 0)
+			(type default)
+		)
+	)
+	(wire
+		(pts
 			(xy 69.85 133.35) (xy 82.55 133.35)
 		)
@@
 	(wire
 		(pts
-			(xy 44.45 106.68) (xy 57.15 106.68)
+			(xy 44.45 106.68) (xy 48.26 106.68)
 		)
 		(stroke
@@
 	(wire
 		(pts
-			(xy 44.45 133.35) (xy 57.15 133.35)
+			(xy 44.45 133.35) (xy 46.99 133.35)
 		)
 		(stroke
@@
 	(wire
 		(pts
+			(xy 46.99 133.35) (xy 57.15 133.35)
+		)
+		(stroke
+			(width 0)
+			(type default)
+		)
+	)
+	(wire
+		(pts
 			(xy 98.425 76.835) (xy 97.79 76.835)
 		)
@@
 	(wire
 		(pts
+			(xy 48.26 106.68) (xy 57.15 106.68)
+		)
+		(stroke
+			(width 0)
+			(type default)
+		)
+	)
+	(wire
+		(pts
 			(xy 114.3 72.39) (xy 121.92 72.39)
 		)
@@
 	)
 	(symbol
+		(lib_id "power:+5V")
+		(at 48.26 104.14 0)
+		(unit 1)
+		(exclude_from_sim no)
+		(in_bom yes)
+		(on_board yes)
+		(dnp no)
+		(property "Reference" "#PWR020"
+			(at 48.26 107.95 0)
+			(effects
+				(font
+					(size 1.27 1.27)
+				)
+				(hide yes)
+			)
+		)
+		(property "Value" "V_BAT+"
+			(at 48.26 100.33 0)
+			(effects
+				(font
+					(size 1.27 1.27)
+				)
+			)
+		)
+		(property "Footprint" ""
+			(at 48.26 104.14 0)
+			(effects
+				(font
+					(size 1.27 1.27)
+				)
+				(hide yes)
+			)
+		)
+		(property "Datasheet" ""
+			(at 48.26 104.14 0)
+			(effects
+				(font
+					(size 1.27 1.27)
+				)
+				(hide yes)
+			)
+		)
+		(property "Description" ""
+			(at 48.26 104.14 0)
+			(effects
+				(font
+					(size 1.27 1.27)
+				)
+				(hide yes)
+			)
+		)
+		(pin "1"
+		)
+		(instances
+			(project "EVAL_TOLT_DC48V_3KW"
+				(path "/ab32ac57-1c18-4307-8f91-d2778314d165/8b314924-91f0-419d-ab10-67cac4e4e0de"
+					(reference "#PWR020")
+					(unit 1)
+				)
+			)
+		)
+	)
+	(symbol
 		(lib_id "C18:100ZLJ820M18X40")
 		(at 107.95 123.19 90)
@@
 					(unit 1)
 				)
+			)
+		)
+	)
+	(symbol
+		(lib_id "power:+5V")
+		(at 46.99 135.89 180)
+		(unit 1)
+		(exclude_from_sim no)
+		(in_bom yes)
+		(on_board yes)
+		(dnp no)
+		(property "Reference" "#PWR021"
+			(at 46.99 132.08 0)
+			(effects
+				(font
+					(size 1.27 1.27)
+				)
+				(hide yes)
+			)
+		)
+		(property "Value" "V_BAT-"
+			(at 46.99 139.7 0)
+			(effects
+				(font
+					(size 1.27 1.27)
+				)
+			)
+		)
+		(property "Footprint" ""
+			(at 46.99 135.89 0)
+			(effects
+				(font
+					(size 1.27 1.27)
+				)
+				(hide yes)
+			)
+		)
+		(property "Datasheet" ""
+			(at 46.99 135.89 0)
+			(effects
+				(font
+					(size 1.27 1.27)
+				)
+				(hide yes)
+			)
+		)
+		(property "Description" ""
+			(at 46.99 135.89 0)
+			(effects
+				(font
+					(size 1.27 1.27)
+				)
+				(hide yes)
+			)
+		)
+		(pin "1"
+		)
+		(instances
+			(project "EVAL_TOLT_DC48V_3KW"
+				(path "/ab32ac57-1c18-4307-8f91-d2778314d165/8b314924-91f0-419d-ab10-67cac4e4e0de"
+					(reference "#PWR021")
+					(unit 1)
+				)

Commit message: v06112024
Parts:
- C20, C21, C22, C23, C24, C25, C26, C89: footprint Kap-1206-Footprints:C20 -> Capacitor_SMD:C_1206_3216Metric
- C60, C62, C63: footprint Kap-1206-Footprints:C8 -> Capacitor_SMD:C_1206_3216Metric
- C61: footprint Kap-1206-Footprints:C15 -> Capacitor_SMD:C_1206_3216Metric
- R42, R46: footprint Resistor-1206-Footprints:R42 -> Resistor_SMD:R_1206_3216Metric_Pad1.30x1.75mm_HandSolder
- R43, R44: footprint Resistor-1206-Footprints:R43 -> Resistor_SMD:R_1206_3216Metric_Pad1.30x1.75mm_HandSolder
- R45: footprint Resistor-1206-Footprints:R12 -> Resistor_SMD:R_1206_3216Metric_Pad1.30x1.75mm_HandSolder
- R47: footprint Resistor-1206-Footprints:R47 -> Resistor_SMD:R_1206_3216Metric_Pad1.30x1.75mm_HandSolder
- R7: footprint Resistor-1206-Footprints:R7 -> Resistor_SMD:R_1206_3216Metric_Pad1.30x1.75mm_HandSolder
Changed lines of the file:
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@@
 			)
 		)
-		(property "Footprint" "Resistor-1206-Footprints:R7"
+		(property "Footprint" "Resistor_SMD:R_1206_3216Metric_Pad1.30x1.75mm_HandSolder"
 			(at 109.982 168.91 90)
 			(effects
@@
 			)
 		)
-		(property "Footprint" "Kap-1206-Footprints:C20"
+		(property "Footprint" "Capacitor_SMD:C_1206_3216Metric"
 			(at 200.66 122.2248 0)
 			(effects
@@
 			)
 		)
-		(property "Footprint" "Kap-1206-Footprints:C8"
+		(property "Footprint" "Capacitor_SMD:C_1206_3216Metric"
 			(at 107.6452 76.2 0)
 			(effects
@@
 			)
 		)
-		(property "Footprint" "Kap-1206-Footprints:C20"
+		(property "Footprint" "Capacitor_SMD:C_1206_3216Metric"
 			(at 162.56 122.2248 0)
 			(effects
@@
 			)
 		)
-		(property "Footprint" "Kap-1206-Footprints:C20"
+		(property "Footprint" "Capacitor_SMD:C_1206_3216Metric"
 			(at 187.96 122.2248 0)
 			(effects
@@
 			)
 		)
-		(property "Footprint" "Kap-1206-Footprints:C20"
+		(property "Footprint" "Capacitor_SMD:C_1206_3216Metric"
 			(at 149.86 122.2248 0)
 			(effects
@@
 			)
 		)
-		(property "Footprint" "Kap-1206-Footprints:C15"
+		(property "Footprint" "Capacitor_SMD:C_1206_3216Metric"
 			(at 127 53.6448 0)
 			(effects
@@
 			)
 		)
-		(property "Footprint" "Resistor-1206-Footprints:R42"
+		(property "Footprint" "Resistor_SMD:R_1206_3216Metric_Pad1.30x1.75mm_HandSolder"
 			(at 77.978 39.37 90)
 			(effects
@@
 			)
 		)
-		(property "Footprint" "Kap-1206-Footprints:C20"
+		(property "Footprint" "Capacitor_SMD:C_1206_3216Metric"
 			(at 124.46 122.2248 0)
 			(effects
@@
 			)
 		)
-		(property "Footprint" "Kap-1206-Footprints:C20"
+		(property "Footprint" "Capacitor_SMD:C_1206_3216Metric"
 			(at 137.16 122.2248 0)
 			(effects
@@
 			)
 		)
-		(property "Footprint" "Resistor-1206-Footprints:R43"
+		(property "Footprint" "Resistor_SMD:R_1206_3216Metric_Pad1.30x1.75mm_HandSolder"
 			(at 61.722 46.99 90)
 			(effects
@@
 			)
 		)
-		(property "Footprint" "Kap-1206-Footprints:C8"
+		(property "Footprint" "Capacitor_SMD:C_1206_3216Metric"
 			(at 83.82 59.9948 0)
 			(effects
@@
 			)
 		)
-		(property "Footprint" "Kap-1206-Footprints:C8"
+		(property "Footprint" "Capacitor_SMD:C_1206_3216Metric"
 			(at 165.1 71.4248 0)
 			(effects
@@
 			)
 		)
-		(property "Footprint" "Resistor-1206-Footprints:R42"
+		(property "Footprint" "Resistor_SMD:R_1206_3216Metric_Pad1.30x1.75mm_HandSolder"
 			(at 118.618 81.28 90)
 			(effects
@@
 			)
 		)
-		(property "Footprint" "Resistor-1206-Footprints:R43"
+		(property "Footprint" "Resistor_SMD:R_1206_3216Metric_Pad1.30x1.75mm_HandSolder"
 			(at 60.452 66.04 90)
 			(effects
@@
 			)
 		)
-		(property "Footprint" "Resistor-1206-Footprints:R47"
+		(property "Footprint" "Resistor_SMD:R_1206_3216Metric_Pad1.30x1.75mm_HandSolder"
 			(at 136.652 60.96 90)
 			(effects
@@
 			)
 		)
-		(property "Footprint" "Resistor-1206-Footprints:R12"
+		(property "Footprint" "Resistor_SMD:R_1206_3216Metric_Pad1.30x1.75mm_HandSolder"
 			(at 110.49 39.878 90)
 			(effects
@@
 			)
 		)
-		(property "Footprint" "Kap-1206-Footprints:C20"
+		(property "Footprint" "Capacitor_SMD:C_1206_3216Metric"
 			(at 213.36 122.2248 0)
 			(effects
@@
 			)
 		)
-		(property "Footprint" "Kap-1206-Footprints:C20"
+		(property "Footprint" "Capacitor_SMD:C_1206_3216Metric"
 			(at 175.26 122.2248 0)
 			(effects

Commit message: v08112024
Connections:
- net I_PHASE_U: now reaches C62.2, OP1.1 (OUT), R46.2, R47.1
Changed lines of the file:
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@@
+		)
+	)
+	(global_label "I_PHASE_U"
+		(shape input)
+		(at 133.35 60.96 90)
+		(fields_autoplaced yes)
+		(effects
+			(font
+				(size 1.27 1.27)
+			)
+			(justify left)
+		)
+		(property "Intersheetrefs" "${INTERSHEET_REFS}"
+			(at 133.35 48.0567 90)
+			(effects
+				(font
+					(size 1.27 1.27)
+				)
+				(justify left)
+				(hide yes)
+			)
 		)
 	)

Commit message: v10112024-2
Other:
- moved on the sheet: OP1

Commit message: v15112024
Changed lines of the file:
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@@
 	)
 	(junction
+		(at 96.774 60.96)
+		(diameter 0)
+		(color 0 0 0 0)
+	)
+	(junction
 		(at 46.99 133.35)
 		(diameter 0)
@@
 	)
 	(junction
+		(at 96.774 63.5)
+		(diameter 0)
+		(color 0 0 0 0)
+	)
+	(junction
 		(at 95.25 133.35)
 		(diameter 0)
@@
 	(wire
 		(pts
-			(xy 91.44 60.96) (xy 101.6 60.96)
+			(xy 91.44 60.96) (xy 96.774 60.96)
+		)
+		(stroke
+			(width 0)
+			(type default)
+		)
+	)
+	(wire
+		(pts
+			(xy 96.774 60.96) (xy 101.6 60.96)
 		)
 		(stroke
@@
 	(wire
 		(pts
-			(xy 91.44 63.5) (xy 101.6 63.5)
+			(xy 91.44 63.5) (xy 96.774 63.5)
 		)
 		(stroke
@@
 	(wire
 		(pts
+			(xy 96.774 63.5) (xy 101.6 63.5)
+		)
+		(stroke
+			(width 0)
+			(type default)
+		)
+	)
+	(wire
+		(pts
 			(xy 120.65 133.35) (xy 133.35 133.35)
 		)
@@
 	)
 	(symbol
+		(lib_id "power:PWR_FLAG")
+		(at 96.774 60.96 0)
+		(unit 1)
+		(exclude_from_sim no)
+		(in_bom yes)
+		(on_board yes)
+		(dnp no)
+		(fields_autoplaced yes)
+		(property "Reference" "#FLG07"
+			(at 96.774 59.055 0)
+			(effects
+				(font
+					(size 1.27 1.27)
+				)
+				(hide yes)
+			)
+		)
+		(property "Value" "PWR_FLAG"
+			(at 96.774 56.134 0)
+			(effects
+				(font
+					(size 1.27 1.27)
+				)
+			)
+		)
+		(property "Footprint" ""
+			(at 96.774 60.96 0)
+			(effects
+				(font
+					(size 1.27 1.27)
+				)
+				(hide yes)
+			)
+		)
+		(property "Datasheet" "~"
+			(at 96.774 60.96 0)
+			(effects
+				(font
+					(size 1.27 1.27)
+				)
+				(hide yes)
+			)
+		)
+		(property "Description" ""
+			(at 96.774 60.96 0)
+			(effects
+				(font
+					(size 1.27 1.27)
+				)
+				(hide yes)
+			)
+		)
+		(pin "1"
+		)
+		(instances
+			(project "EVAL_TOLT_DC48V_3KW"
+				(path "/ab32ac57-1c18-4307-8f91-d2778314d165/8b314924-91f0-419d-ab10-67cac4e4e0de"
+					(reference "#FLG07")
+					(unit 1)
+				)
+			)
+		)
+	)
+	(symbol
 		(lib_id "power:GNDREF")
 		(at 69.85 144.78 0)
@@
 					(unit 1)
 				)
+			)
+		)
+	)
+	(symbol
+		(lib_id "power:PWR_FLAG")
+		(at 96.774 63.5 180)
+		(unit 1)
+		(exclude_from_sim no)
+		(in_bom yes)
+		(on_board yes)
+		(dnp no)
+		(fields_autoplaced yes)
+		(property "Reference" "#FLG08"
+			(at 96.774 65.405 0)
+			(effects
+				(font
+					(size 1.27 1.27)
+				)
+				(hide yes)
+			)
+		)
+		(property "Value" "PWR_FLAG"
+			(at 96.774 68.58 0)
+			(effects
+				(font
+					(size 1.27 1.27)
+				)
+			)
+		)
+		(property "Footprint" ""
+			(at 96.774 63.5 0)
+			(effects
+				(font
+					(size 1.27 1.27)
+				)
+				(hide yes)
+			)
+		)
+		(property "Datasheet" "~"
+			(at 96.774 63.5 0)
+			(effects
+				(font
+					(size 1.27 1.27)
+				)
+				(hide yes)
+			)
+		)
+		(property "Description" ""
+			(at 96.774 63.5 0)
+			(effects
+				(font
+					(size 1.27 1.27)
+				)
+				(hide yes)
+			)
+		)
+		(pin "1"
+		)
+		(instances
+			(project "EVAL_TOLT_DC48V_3KW"
+				(path "/ab32ac57-1c18-4307-8f91-d2778314d165/8b314924-91f0-419d-ab10-67cac4e4e0de"
+					(reference "#FLG08")
+					(unit 1)
+				)
