File: EVAL-TOLT-DC48V-3KW-TOBO2-1206/Power Board Connector.kicad_sch (KiCad schematic)
At the start: 23 parts, among them J12 Direction Switch, Q7 IRLML6346, U12 PCN10-32S-2.54DSA72

Commit message: v06112024
Parts:
- C80: footprint Kap-1206-Footprints:C15 -> Capacitor_SMD:C_1206_3216Metric
- C81, C811, C82, C821: footprint Kap-1206-Footprints:C72 -> Capacitor_SMD:C_1206_3216Metric
- R72, R78, R79: footprint Resistor-1206-Footprints:R72 -> Resistor_SMD:R_1206_3216Metric_Pad1.30x1.75mm_HandSolder
- R73: footprint Resistor-1206-Footprints:R13 -> Resistor_SMD:R_1206_3216Metric_Pad1.30x1.75mm_HandSolder
- R74: footprint Resistor-1206-Footprints:R74 -> Resistor_SMD:R_1206_3216Metric_Pad1.30x1.75mm_HandSolder
- R75, R751: footprint Resistor-1206-Footprints:R75 -> Resistor_SMD:R_1206_3216Metric_Pad1.30x1.75mm_HandSolder
- R76, R762: footprint Resistor-1206-Footprints:R76 -> Resistor_SMD:R_1206_3216Metric_Pad1.30x1.75mm_HandSolder
- R77: footprint Resistor-1206-Footprints:R77 -> Resistor_SMD:R_1206_3216Metric_Pad1.30x1.75mm_HandSolder
- R80: footprint Resistor-1206-Footprints:R7 -> Resistor_SMD:R_1206_3216Metric_Pad1.30x1.75mm_HandSolder
Changed lines of the file:
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@@
 			)
 		)
-		(property "Footprint" "Resistor-1206-Footprints:R75"
+		(property "Footprint" "Resistor_SMD:R_1206_3216Metric_Pad1.30x1.75mm_HandSolder"
 			(at 228.6 21.717 90)
 			(effects
@@
 			)
 		)
-		(property "Footprint" "Resistor-1206-Footprints:R7"
+		(property "Footprint" "Resistor_SMD:R_1206_3216Metric_Pad1.30x1.75mm_HandSolder"
 			(at 220.472 124.46 90)
 			(effects
@@
 			)
 		)
-		(property "Footprint" "Resistor-1206-Footprints:R13"
+		(property "Footprint" "Resistor_SMD:R_1206_3216Metric_Pad1.30x1.75mm_HandSolder"
 			(at 26.67 76.708 90)
 			(effects
@@
 			)
 		)
-		(property "Footprint" "Resistor-1206-Footprints:R75"
+		(property "Footprint" "Resistor_SMD:R_1206_3216Metric_Pad1.30x1.75mm_HandSolder"
 			(at 222.25 61.722 90)
 			(effects
@@
 			)
 		)
-		(property "Footprint" "Resistor-1206-Footprints:R72"
+		(property "Footprint" "Resistor_SMD:R_1206_3216Metric_Pad1.30x1.75mm_HandSolder"
 			(at 196.85 123.698 90)
 			(effects
@@
 			)
 		)
-		(property "Footprint" "Kap-1206-Footprints:C72"
+		(property "Footprint" "Capacitor_SMD:C_1206_3216Metric"
 			(at 355.27 85.09 0)
 			(effects
@@
 			)
 		)
-		(property "Footprint" "Resistor-1206-Footprints:R74"
+		(property "Footprint" "Resistor_SMD:R_1206_3216Metric_Pad1.30x1.75mm_HandSolder"
 			(at 26.67 104.648 90)
 			(effects
@@
 			)
 		)
-		(property "Footprint" "Kap-1206-Footprints:C15"
+		(property "Footprint" "Capacitor_SMD:C_1206_3216Metric"
 			(at 52.07 102.87 0)
 			(effects
@@
 			)
 		)
-		(property "Footprint" "Resistor-1206-Footprints:R77"
+		(property "Footprint" "Resistor_SMD:R_1206_3216Metric_Pad1.30x1.75mm_HandSolder"
 			(at 180.34 111.252 90)
 			(effects
@@
 			)
 		)
-		(property "Footprint" "Kap-1206-Footprints:C72"
+		(property "Footprint" "Capacitor_SMD:C_1206_3216Metric"
 			(at 355.27 44.45 0)
 			(effects
@@
 			)
 		)
-		(property "Footprint" "Resistor-1206-Footprints:R72"
+		(property "Footprint" "Resistor_SMD:R_1206_3216Metric_Pad1.30x1.75mm_HandSolder"
 			(at 54.61 31.242 90)
 			(effects
@@
 			)
 		)
-		(property "Footprint" "Resistor-1206-Footprints:R76"
+		(property "Footprint" "Resistor_SMD:R_1206_3216Metric_Pad1.30x1.75mm_HandSolder"
 			(at 192.278 74.93 90)
 			(effects
@@
 			)
 		)
-		(property "Footprint" "Kap-1206-Footprints:C72"
+		(property "Footprint" "Capacitor_SMD:C_1206_3216Metric"
 			(at 68.91 54.61 0)
 			(effects
@@
 			)
 		)
-		(property "Footprint" "Resistor-1206-Footprints:R72"
+		(property "Footprint" "Resistor_SMD:R_1206_3216Metric_Pad1.30x1.75mm_HandSolder"
 			(at 210.82 124.968 90)
 			(effects
@@
 			)
 		)
-		(property "Footprint" "Resistor-1206-Footprints:R76"
+		(property "Footprint" "Resistor_SMD:R_1206_3216Metric_Pad1.30x1.75mm_HandSolder"
 			(at 192.278 66.04 90)
 			(effects
@@
 			)
 		)
-		(property "Footprint" "Kap-1206-Footprints:C72"
+		(property "Footprint" "Capacitor_SMD:C_1206_3216Metric"
 			(at 53.67 54.61 0)
 			(effects

Commit message: v07112024
Connections:
- net +BATT renamed V_BATT+
Changed lines of the file:
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@@
 		(on_board yes)
 		(dnp no)
-		(fields_autoplaced yes)
 		(property "Reference" "#PWR077"
 			(at 26.67 58.42 0)
@@
 			)
 		)
-		(property "Value" "+BATT"
-			(at 26.67 50.8 0)
+		(property "Value" "V_BATT+"
+			(at 22.606 49.784 0)
 			(effects
 				(font
 					(size 1.27 1.27)
 				)
+				(justify left)
 			)
 		)

Commit message: v08112024
Connections:
- net V_BATT+ renamed V_BAT+
Changed lines of the file:
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@@
 			)
 		)
-		(property "Value" "V_BATT+"
+		(property "Value" "V_BAT+"
 			(at 22.606 49.784 0)
 			(effects

Commit message: v10112024
Parts:
- D15: footprint Misc-Footprints:D15 -> Diode_SMD:D_1206_3216Metric_Pad1.42x1.75mm_HandSolder
- U12: footprint Misc-Footprints:PCN -> Connector_IDC:IDC-Header_2x17_P2.54mm_Vertical
Changed lines of the file:
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@@
 			)
 		)
-		(property "Footprint" "Misc-Footprints:PCN"
+		(property "Footprint" "Connector_IDC:IDC-Header_2x17_P2.54mm_Vertical"
 			(at 154.94 114.3 0)
 			(effects
@@
 			)
 		)
-		(property "Footprint" "Misc-Footprints:D15"
+		(property "Footprint" "Diode_SMD:D_1206_3216Metric_Pad1.42x1.75mm_HandSolder"
 			(at 68.58 99.06 0)
 			(effects

Commit message: v10112024-2
Parts:
- J12: footprint Misc-Footprints:J12 -> Connector_PinHeader_2.54mm:PinHeader_1x02_P2.54mm_Vertical; symbol TSW-102-08-L-S:TSW-102-08-L-S -> PCM_SL_Pin_Headers:PINHD_1x2_Male
Connections:
- net GNDS: now also C82.1, J12.1, RT1.3 (GND); no longer C82.2, J12.01, R75.1, RT1.1 (V_{DD})
- net at R72.1: now also J12.2; no longer J12.02
- new net: C82.2, R75.1, RT1.1 (V_{DD})

Commit message: v15112024
Parts:
- D15: footprint Diode_SMD:D_1206_3216Metric_Pad1.42x1.75mm_HandSolder -> Misc-Footprints:DO-214AA
- J12: footprint Connector_PinHeader_2.54mm:PinHeader_1x02_P2.54mm_Vertical -> Misc-Footprints:TSW-102-XX-YY-S
- U12: footprint Connector_IDC:IDC-Header_2x17_P2.54mm_Vertical -> Connector_IDC:IDC-Header_2x15_P2.54mm_Vertical
Connections:
- net +5V: now also U12.4, U12.6; no longer U12.16, U12.32
- net BEMF_PHASE_U: now also U12.8; no longer U12.20
- net DR_EN: now also U12.12; no longer U12.31
- net I_SNS_PHASE_U: now also U12.7; no longer U12.5
- net U-H: now also U12.11; no longer U12.25
- net U-L: now also U12.9; no longer U12.24
- net at U12.10: now also C811.2, R762.1
- net at U12.13: now also C80.2, D15.1 (K), R73.1, R74.1
- net at C81.2, R76.1: now also U12.5; no longer U12.8
- now unconnected: U12.19
Changed lines of the file:
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@@
 	)
 	(junction
+		(at 193.548 134.62)
+		(diameter 0)
+		(color 0 0 0 0)
+	)
+	(junction
 		(at 68.58 88.392)
 		(diameter 0)
@@
 	)
 	(no_connect
-		(at 99.06 114.3)
+		(at 76.2 114.3)
 	)
 	(no_connect
-		(at 101.6 114.3)
+		(at 93.98 114.3)
 	)
 	(no_connect
-		(at 129.54 114.3)
+		(at 99.06 114.3)
 	)
 	(no_connect
-		(at 83.82 114.3)
+		(at 121.92 114.3)
 	)
 	(no_connect
-		(at 147.32 114.3)
+		(at 83.82 114.3)
 	)
 	(no_connect
-		(at 121.92 114.3)
+		(at 114.3 114.3)
 	)
 	(no_connect
-		(at 86.36 114.3)
+		(at 91.44 114.3)
 	)
 	(no_connect
-		(at 111.76 114.3)
+		(at 88.9 114.3)
 	)
 	(no_connect
-		(at 142.24 114.3)
+		(at 116.84 114.3)
 	)
 	(no_connect
-		(at 139.7 114.3)
+		(at 104.14 114.3)
 	)
 	(no_connect
-		(at 127 114.3)
+		(at 78.74 114.3)
 	)
 	(no_connect
-		(at 91.44 114.3)
+		(at 96.52 114.3)
 	)
 	(no_connect
@@
 	)
 	(no_connect
-		(at 104.14 114.3)
+		(at 109.22 114.3)
 	)
 	(no_connect
-		(at 132.08 114.3)
+		(at 111.76 114.3)
 	)
 	(no_connect
-		(at 88.9 114.3)
+		(at 86.36 114.3)
 	)
 	(no_connect
-		(at 114.3 114.3)
+		(at 106.68 114.3)
 	)
 	(no_connect
-		(at 124.46 114.3)
+		(at 101.6 114.3)
 	)
 	(wire
@@
 	(wire
 		(pts
-			(xy 68.58 87.63) (xy 68.58 88.392)
+			(xy 68.58 88.392) (xy 124.46 88.392)
 		)
 		(stroke
@@
 	(wire
 		(pts
-			(xy 134.62 66.04) (xy 165.1 66.04)
+			(xy 259.08 93.98) (xy 259.08 100.33)
 		)
 		(stroke
@@
 	(wire
 		(pts
-			(xy 259.08 93.98) (xy 259.08 100.33)
+			(xy 52.07 88.392) (xy 68.58 88.392)
 		)
 		(stroke
@@
 	(wire
 		(pts
-			(xy 52.07 88.392) (xy 68.58 88.392)
+			(xy 196.85 97.79) (xy 210.82 97.79)
 		)
 		(stroke
@@
 	(wire
 		(pts
-			(xy 137.16 74.93) (xy 137.16 114.3)
+			(xy 180.34 134.62) (xy 193.548 134.62)
 		)
 		(stroke
@@
 	(wire
 		(pts
-			(xy 196.85 97.79) (xy 210.82 97.79)
+			(xy 190.5 57.15) (xy 233.68 57.15)
 		)
 		(stroke
@@
 	(wire
 		(pts
-			(xy 180.34 134.62) (xy 202.692 134.62)
+			(xy 142.24 114.3) (xy 142.24 30.48)
 		)
 		(stroke
@@
 	(wire
 		(pts
-			(xy 190.5 57.15) (xy 233.68 57.15)
+			(xy 144.78 74.93) (xy 149.86 74.93)
 		)
 		(stroke
@@
 	(wire
 		(pts
-			(xy 210.312 124.46) (xy 210.82 124.46)
+			(xy 193.548 134.62) (xy 202.692 134.62)
 		)
 		(stroke
@@
 	(wire
 		(pts
-			(xy 152.4 106.68) (xy 152.4 114.3)
+			(xy 210.312 124.46) (xy 210.82 124.46)
 		)
 		(stroke
@@
 	(wire
 		(pts
-			(xy 165.1 99.06) (xy 165.1 134.62)
+			(xy 152.4 106.68) (xy 152.4 114.3)
 		)
 		(stroke
@@
 	(wire
 		(pts
-			(xy 109.22 87.63) (xy 109.22 114.3)
+			(xy 165.1 99.06) (xy 165.1 134.62)
 		)
 		(stroke
@@
 	(wire
 		(pts
-			(xy 210.312 124.46) (xy 210.312 129.54)
+			(xy 132.08 66.04) (xy 165.1 66.04)
 		)
 		(stroke
@@
 	(wire
 		(pts
-			(xy 68.58 87.63) (xy 109.22 87.63)
+			(xy 210.312 124.46) (xy 210.312 129.54)
 		)
 		(stroke
@@
 	(wire
 		(pts
-			(xy 134.62 114.3) (xy 134.62 66.04)
-		)
-		(stroke
-			(width 0)
-			(type default)
-		)
-	)
-	(wire
-		(pts
 			(xy 207.01 74.93) (xy 190.5 74.93)
 		)
@@
 	(wire
 		(pts
-			(xy 137.16 74.93) (xy 149.86 74.93)
-		)
-		(stroke
-			(width 0)
-			(type default)
-		)
-	)
-	(wire
-		(pts
-			(xy 144.78 99.06) (xy 144.78 114.3)
-		)
-		(stroke
-			(width 0)
-			(type default)
-		)
-	)
-	(wire
-		(pts
 			(xy 259.08 54.61) (xy 259.08 55.88)
 		)
@@
 	(wire
 		(pts
-			(xy 76.2 30.48) (xy 54.61 30.48)
+			(xy 54.61 30.48) (xy 142.24 30.48)
 		)
 		(stroke
@@
 	(wire
 		(pts
-			(xy 78.74 104.14) (xy 78.74 114.3)
+			(xy 124.46 88.392) (xy 124.46 114.3)
 		)
 		(stroke
@@
 	(wire
 		(pts
-			(xy 106.68 111.76) (xy 106.68 114.3)
+			(xy 132.08 66.04) (xy 132.08 114.3)
 		)
 		(stroke
@@
 	(wire
 		(pts
+			(xy 144.78 74.93) (xy 144.78 114.3)
+		)
+		(stroke
+			(width 0)
+			(type default)
+		)
+	)
+	(wire
+		(pts
 			(xy 259.08 53.34) (xy 259.08 54.61)
 		)
@@
 	(wire
 		(pts
-			(xy 76.2 114.3) (xy 76.2 30.48)
-		)
-		(stroke
-			(width 0)
-			(type default)
-		)
-	)
-	(wire
-		(pts
 			(xy 223.012 91.44) (xy 223.012 88.392)
 		)
@@
 	)
 	(label "DR_EN"
-		(at 78.74 104.14 90)
+		(at 127 114.3 90)
 		(fields_autoplaced yes)
 		(effects
@@
 	(global_label "BEMF_PHASE_U"
 		(shape input)
-		(at 106.68 111.76 90)
+		(at 137.16 114.3 90)
 		(fields_autoplaced yes)
 		(effects
@@
 		)
 		(property "Intersheetrefs" "${INTERSHEET_REFS}"
-			(at 106.68 94.5025 90)
+			(at 137.16 97.0425 90)
 			(effects
 				(font
@@
 	(global_label "U-H"
 		(shape input)
-		(at 93.98 114.3 90)
+		(at 129.54 114.3 90)
 		(fields_autoplaced yes)
 		(effects
@@
 		)
 		(property "Intersheetrefs" "${INTERSHEET_REFS}"
-			(at 93.98 107.0814 90)
+			(at 129.54 107.0814 90)
 			(effects
 				(font
@@
 	(global_label "U-L"
 		(shape input)
-		(at 96.52 114.3 90)
+		(at 134.62 114.3 90)
 		(fields_autoplaced yes)
 		(effects
@@
 		)
 		(property "Intersheetrefs" "${INTERSHEET_REFS}"
-			(at 96.52 107.3838 90)
+			(at 134.62 107.3838 90)
 			(effects
 				(font
@@
 	(global_label "I_SNS_PHASE_U"
 		(shape input)
-		(at 144.78 99.06 90)
+		(at 139.7 114.3 90)
 		(fields_autoplaced yes)
 		(effects
@@
 		)
 		(property "Intersheetrefs" "${INTERSHEET_REFS}"
-			(at 144.78 81.4396 90)
+			(at 139.7 96.6796 90)
 			(effects
 				(font
@@
 			)
 		)
-		(property "Footprint" "Connector_IDC:IDC-Header_2x17_P2.54mm_Vertical"
+		(property "Footprint" "Connector_IDC:IDC-Header_2x15_P2.54mm_Vertical"
 			(at 154.94 114.3 0)
 			(effects
@@
 			)
 		)
-		(property "Footprint" "Diode_SMD:D_1206_3216Metric_Pad1.42x1.75mm_HandSolder"
+		(property "Footprint" "Misc-Footprints:DO-214AA"
 			(at 68.58 99.06 0)
 			(effects
@@
 			)
 		)
-		(property "Footprint" "Connector_PinHeader_2.54mm:PinHeader_1x02_P2.54mm_Vertical"
+		(property "Footprint" "Misc-Footprints:TSW-102-XX-YY-S"
 			(at 49.53 50.292 0)
 			(effects
@@
 	(symbol
 		(lib_id "power:+5V")
-		(at 116.84 114.3 0)
+		(at 147.32 114.3 0)
 		(unit 1)
 		(exclude_from_sim no)
@@
 		(dnp no)
 		(property "Reference" "#PWR010"
-			(at 116.84 118.11 0)
+			(at 147.32 118.11 0)
 			(effects
 				(font
@@
 		)
 		(property "Value" "+5V"
-			(at 116.586 111.252 90)
+			(at 147.066 111.252 90)
 			(effects
 				(font
@@
 		)
 		(property "Footprint" ""
-			(at 116.84 114.3 0)
+			(at 147.32 114.3 0)
 			(effects
 				(font
@@
 		)
 		(property "Datasheet" ""
-			(at 116.84 114.3 0)
+			(at 147.32 114.3 0)
 			(effects
 				(font
@@
 		)
 		(property "Description" ""
-			(at 116.84 114.3 0)
+			(at 147.32 114.3 0)
 			(effects
 				(font
@@
 					(unit 1)
 				)
+			)
+		)
+	)
+	(symbol
+		(lib_id "power:PWR_FLAG")
+		(at 193.548 134.62 180)
+		(unit 1)
+		(exclude_from_sim no)
+		(in_bom yes)
+		(on_board yes)
+		(dnp no)
+		(fields_autoplaced yes)
+		(property "Reference" "#FLG017"
+			(at 193.548 136.525 0)
+			(effects
+				(font
+					(size 1.27 1.27)
+				)
+				(hide yes)
+			)
+		)
+		(property "Value" "PWR_FLAG"
+			(at 193.548 139.192 0)
+			(effects
+				(font
+					(size 1.27 1.27)
+				)
+			)
+		)
+		(property "Footprint" ""
+			(at 193.548 134.62 0)
+			(effects
+				(font
+					(size 1.27 1.27)
+				)
+				(hide yes)
+			)
+		)
+		(property "Datasheet" "~"
+			(at 193.548 134.62 0)
+			(effects
+				(font
+					(size 1.27 1.27)
+				)
+				(hide yes)
+			)
+		)
+		(property "Description" ""
+			(at 193.548 134.62 0)
+			(effects
+				(font
+					(size 1.27 1.27)
+				)
+				(hide yes)
+			)
+		)
+		(pin "1"
+		)
+		(instances
+			(project "EVAL_TOLT_DC48V_3KW"
+				(path "/ab32ac57-1c18-4307-8f91-d2778314d165/c5d2820f-dc5b-4980-906d-0f8bd6a51e5e"
+					(reference "#FLG017")
+					(unit 1)
+				)
