File: EVAL-TOLT-DC48V-3KW-TOBO2-1206/U-Phase.kicad_sch (KiCad schematic)
At the start: 33 parts, among them Q1 IAUS300N10S5N015TATMA1, Q4 IAUS300N10S5N015TATMA1, U3 2EDL8x24G, U4 NL27WZ08USG

Commit message: v06112024
Parts:
- C27: footprint Kap-1206-Footprints:C1 -> Capacitor_SMD:C_1206_3216Metric
- C28, C29: footprint Kap-1206-Footprints:C28 -> Capacitor_SMD:C_1206_3216Metric
- C30: footprint Kap-1206-Footprints:C30 -> Capacitor_SMD:C_1206_3216Metric
- C31, C32: footprint Kap-1206-Footprints:C31 -> Capacitor_SMD:C_1206_3216Metric
- C35: footprint Kap-1206-Footprints:C35 -> Capacitor_SMD:C_1206_3216Metric
- C36: footprint Kap-1206-Footprints:C36 -> Capacitor_SMD:C_1206_3216Metric
- C37: footprint Kap-1206-Footprints:C15 -> Capacitor_SMD:C_1206_3216Metric
- C83, C84: footprint Kap-1206-Footprints:C83 -> Capacitor_SMD:C_1206_3216Metric
- C94: footprint Kap-1206-Footprints:C94 -> Capacitor_SMD:C_1206_3216Metric
- R10, R15: footprint Resistor-1206-Footprints:R10 -> Resistor_SMD:R_1206_3216Metric_Pad1.30x1.75mm_HandSolder
- R11, R16: footprint Resistor-1206-Footprints:R11 -> Resistor_SMD:R_1206_3216Metric_Pad1.30x1.75mm_HandSolder
- R12, R18: footprint Resistor-1206-Footprints:R12 -> Resistor_SMD:R_1206_3216Metric_Pad1.30x1.75mm_HandSolder
- R13, R19: footprint Resistor-1206-Footprints:R13 -> Resistor_SMD:R_1206_3216Metric_Pad1.30x1.75mm_HandSolder
- R14: footprint Resistor-1206-Footprints:R14 -> Resistor_SMD:R_1206_3216Metric_Pad1.30x1.75mm_HandSolder
- R17: footprint Resistor-1206-Footprints:R17 -> Resistor_SMD:R_1206_3216Metric_Pad1.30x1.75mm_HandSolder
- R81, R82: footprint Resistor-1206-Footprints:R47 -> Resistor_SMD:R_1206_3216Metric_Pad1.30x1.75mm_HandSolder
Connections:
- net +BATT renamed V_BAT+
Changed lines of the file:
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@@
 			)
 		)
-		(property "Footprint" "Resistor-1206-Footprints:R13"
+		(property "Footprint" "Resistor_SMD:R_1206_3216Metric_Pad1.30x1.75mm_HandSolder"
 			(at 151.13 106.172 90)
 			(effects
@@
 			)
 		)
-		(property "Footprint" "Resistor-1206-Footprints:R47"
+		(property "Footprint" "Resistor_SMD:R_1206_3216Metric_Pad1.30x1.75mm_HandSolder"
 			(at 31.242 133.35 90)
 			(effects
@@
 			)
 		)
-		(property "Footprint" "Kap-1206-Footprints:C31"
+		(property "Footprint" "Capacitor_SMD:C_1206_3216Metric"
 			(at 236.22 106.68 0)
 			(effects
@@
 			)
 		)
-		(property "Footprint" "Resistor-1206-Footprints:R11"
+		(property "Footprint" "Resistor_SMD:R_1206_3216Metric_Pad1.30x1.75mm_HandSolder"
 			(at 130.048 40.64 90)
 			(effects
@@
 			)
 		)
-		(property "Footprint" "Kap-1206-Footprints:C36"
+		(property "Footprint" "Capacitor_SMD:C_1206_3216Metric"
 			(at 41.91 43.4848 0)
 			(effects
@@
 			)
 		)
-		(property "Footprint" "Kap-1206-Footprints:C31"
+		(property "Footprint" "Capacitor_SMD:C_1206_3216Metric"
 			(at 236.22 59.69 0)
 			(effects
@@
 			)
 		)
-		(property "Footprint" "Kap-1206-Footprints:C94"
+		(property "Footprint" "Capacitor_SMD:C_1206_3216Metric"
 			(at 251.46 54.9148 0)
 			(effects
@@
 			)
 		)
-		(property "Footprint" "Resistor-1206-Footprints:R11"
+		(property "Footprint" "Resistor_SMD:R_1206_3216Metric_Pad1.30x1.75mm_HandSolder"
 			(at 130.048 86.36 90)
 			(effects
@@
 			)
 		)
-		(property "Footprint" "Kap-1206-Footprints:C83"
+		(property "Footprint" "Capacitor_SMD:C_1206_3216Metric"
 			(at 115.57 141.2748 0)
 			(effects
@@
 			)
 		)
-		(property "Footprint" "Resistor-1206-Footprints:R14"
+		(property "Footprint" "Resistor_SMD:R_1206_3216Metric_Pad1.30x1.75mm_HandSolder"
 			(at 252.73 91.948 90)
 			(effects
@@
 			)
 		)
-		(property "Footprint" "Kap-1206-Footprints:C35"
+		(property "Footprint" "Capacitor_SMD:C_1206_3216Metric"
 			(at 107.95 72.6948 0)
 			(effects
@@
 			)
 		)
-		(property "Footprint" "Kap-1206-Footprints:C30"
+		(property "Footprint" "Capacitor_SMD:C_1206_3216Metric"
 			(at 280.67 46.99 0)
 			(effects
@@
 			)
 		)
-		(property "Footprint" "Resistor-1206-Footprints:R17"
+		(property "Footprint" "Resistor_SMD:R_1206_3216Metric_Pad1.30x1.75mm_HandSolder"
 			(at 252.73 103.632 90)
 			(effects
@@
 			)
 		)
-		(property "Footprint" "Resistor-1206-Footprints:R12"
+		(property "Footprint" "Resistor_SMD:R_1206_3216Metric_Pad1.30x1.75mm_HandSolder"
 			(at 126.238 93.98 90)
 			(effects
@@
 			)
 		)
-		(property "Footprint" "Kap-1206-Footprints:C1"
+		(property "Footprint" "Capacitor_SMD:C_1206_3216Metric"
 			(at 256.54 49.53 0)
 			(effects
@@
 			)
 		)
-		(property "Footprint" "Kap-1206-Footprints:C15"
+		(property "Footprint" "Capacitor_SMD:C_1206_3216Metric"
 			(at 69.85 89.2048 0)
 			(effects
@@
 			)
 		)
-		(property "Footprint" "Kap-1206-Footprints:C28"
+		(property "Footprint" "Capacitor_SMD:C_1206_3216Metric"
 			(at 264.16 49.53 0)
 			(effects
@@
 			)
 		)
-		(property "Value" "+BATT"
-			(at 227.965 24.13 0)
+		(property "Value" "V_BAT+"
+			(at 227.965 22.86 0)
 			(effects
 				(font
@@
 			)
 		)
-		(property "Footprint" "Kap-1206-Footprints:C83"
+		(property "Footprint" "Capacitor_SMD:C_1206_3216Metric"
 			(at 54.61 141.2748 0)
 			(effects
@@
 			)
 		)
-		(property "Footprint" "Resistor-1206-Footprints:R13"
+		(property "Footprint" "Resistor_SMD:R_1206_3216Metric_Pad1.30x1.75mm_HandSolder"
 			(at 151.13 59.182 90)
 			(effects
@@
 			)
 		)
-		(property "Footprint" "Resistor-1206-Footprints:R10"
+		(property "Footprint" "Resistor_SMD:R_1206_3216Metric_Pad1.30x1.75mm_HandSolder"
 			(at 236.22 99.568 90)
 			(effects
@@
 			)
 		)
-		(property "Footprint" "Resistor-1206-Footprints:R12"
+		(property "Footprint" "Resistor_SMD:R_1206_3216Metric_Pad1.30x1.75mm_HandSolder"
 			(at 127.508 52.07 90)
 			(effects
@@
 			)
 		)
-		(property "Footprint" "Resistor-1206-Footprints:R47"
+		(property "Footprint" "Resistor_SMD:R_1206_3216Metric_Pad1.30x1.75mm_HandSolder"
 			(at 90.932 133.35 90)
 			(effects
@@
 			)
 		)
-		(property "Footprint" "Resistor-1206-Footprints:R10"
+		(property "Footprint" "Resistor_SMD:R_1206_3216Metric_Pad1.30x1.75mm_HandSolder"
 			(at 236.22 52.578 90)
 			(effects
@@
 			)
 		)
-		(property "Footprint" "Kap-1206-Footprints:C28"
+		(property "Footprint" "Capacitor_SMD:C_1206_3216Metric"
 			(at 273.05 49.53 0)
 			(effects

Commit message: v10112024
Parts:
- D3: footprint Misc-Footprints:D3 -> Diode_SMD:D_1206_3216Metric_Pad1.42x1.75mm_HandSolder
- D4, D5: footprint Misc-Footprints:D4 -> Diode_SMD:D_1206_3216Metric_Pad1.42x1.75mm_HandSolder
Changed lines of the file:
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@@
 		)
 	)
-	(label "U_CS+"
-		(at 93.98 59.69 0)
-		(fields_autoplaced yes)
-		(effects
-			(font
-				(size 1.27 1.27)
-			)
-			(justify left bottom)
-		)
-	)
 	(label "+5V"
 		(at 60.325 83.82 0)
@@
 		)
 	)
+	(global_label "U_CS+"
+		(shape input)
+		(at 93.98 59.69 0)
+		(fields_autoplaced yes)
+		(effects
+			(font
+				(size 1.27 1.27)
+			)
+			(justify left)
+		)
+		(property "Intersheetrefs" "${INTERSHEET_REFS}"
+			(at 103.3152 59.69 0)
+			(effects
+				(font
+					(size 1.27 1.27)
+				)
+				(justify left)
+				(hide yes)
+			)
+		)
+	)
 	(global_label "U-L"
 		(shape input)
@@
 			)
 		)
-		(property "Footprint" "Misc-Footprints:D3"
+		(property "Footprint" "Diode_SMD:D_1206_3216Metric_Pad1.42x1.75mm_HandSolder"
 			(at 85.725 33.02 0)
 			(effects
@@
 			)
 		)
-		(property "Footprint" "Misc-Footprints:D4"
+		(property "Footprint" "Diode_SMD:D_1206_3216Metric_Pad1.42x1.75mm_HandSolder"
 			(at 139.7 93.98 0)
 			(effects
@@
 			)
 		)
-		(property "Footprint" "Misc-Footprints:D4"
+		(property "Footprint" "Diode_SMD:D_1206_3216Metric_Pad1.42x1.75mm_HandSolder"
 			(at 139.7 52.07 0)
 			(effects

Commit message: v11112024-3
Parts:
- Q1, Q4: value IAUS300N10S5N015TATMA1 -> IPTG014N10NM5ATMA1; footprint just-footprints:Q1 -> Misc-Footprints:IPTG210N25NM3FDATMA1; symbol IAUS300N10S5N015T:IAUS300N10S5N015TATMA1 -> IPTG014N10NM5ATMA1:IPTG014N10NM5ATMA1; Height (none) -> 2.5; Manufacturer_Name (none) -> Infineon; Manufacturer_Part_Number (none) -> IPTG014N10NM5ATMA1; Mouser Part Number (none) -> 726-IPTG014N10NM5ATM; Mouser Price/Stock (none) -> https://www.mouser.co.uk/ProductDetail/Infineon-Technologie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
Connections:
- net U: now also Q1.8 (S_7); no longer Q1.1 (SOURCE), Q4.10 (DRAIN), Q4.11 (DRAIN), Q4.12 (DRAIN), Q4.13 (DRAIN), Q4.14 (DRAIN), Q4.15 (DRAIN), Q4.16 (DRAIN)
- net U_CS+: now also Q4.8 (S_7); no longer Q4.1 (SOURCE)
- net V_BAT+: no longer Q1.10 (DRAIN), Q1.11 (DRAIN), Q1.12 (DRAIN), Q1.13 (DRAIN), Q1.14 (DRAIN), Q1.15 (DRAIN), Q1.16 (DRAIN)
- net at D5.2 (A), R16.1, R19.1: now also Q4.1 (G); no longer Q4.8 (GATE)
- net at D4.2 (A), R11.1, R13.1: now also Q1.1 (G); no longer Q1.8 (GATE)
Other:
- moved on the sheet: U3, U4

Commit message: v15112024
Parts:
- D3: footprint Diode_SMD:D_1206_3216Metric_Pad1.42x1.75mm_HandSolder -> Diode_SMD:D_SOD-123F
Connections:
- net U-L: no longer R81.1
- new net U-H: R81.1
Changed lines of the file:
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@@
 	)
 	(junction
+		(at 38.1 47.244)
+		(diameter 0)
+		(color 0 0 0 0)
+	)
+	(junction
 		(at 228.092 35.052)
 		(diameter 0)
@@
 	(wire
 		(pts
+			(xy 38.1 47.244) (xy 38.1 50.8)
+		)
+		(stroke
+			(width 0)
+			(type default)
+		)
+	)
+	(wire
+		(pts
 			(xy 151.13 49.022) (xy 177.292 49.022)
 		)
@@
 	(wire
 		(pts
-			(xy 38.1 44.45) (xy 38.1 50.8)
+			(xy 38.1 44.45) (xy 38.1 47.244)
 		)
 		(stroke
@@
 		)
 	)
-	(global_label "U-L"
+	(global_label "U-H"
 		(shape input)
 		(at 24.13 133.35 180)
@@
 		)
 		(property "Intersheetrefs" "${INTERSHEET_REFS}"
-			(at 17.2932 133.35 0)
+			(at 16.9114 133.35 0)
 			(effects
 				(font
@@
 			)
 		)
-		(property "Footprint" "Diode_SMD:D_1206_3216Metric_Pad1.42x1.75mm_HandSolder"
+		(property "Footprint" "Diode_SMD:D_SOD-123F"
 			(at 85.852 33.02 0)
 			(effects
@@
 					(unit 1)
 				)
+			)
+		)
+	)
+	(symbol
+		(lib_id "power:PWR_FLAG")
+		(at 38.1 47.244 270)
+		(unit 1)
+		(exclude_from_sim no)
+		(in_bom yes)
+		(on_board yes)
+		(dnp no)
+		(fields_autoplaced yes)
+		(property "Reference" "#FLG03"
+			(at 40.005 47.244 0)
+			(effects
+				(font
+					(size 1.27 1.27)
+				)
+				(hide yes)
+			)
+		)
+		(property "Value" "PWR_FLAG"
+			(at 41.402 47.2439 90)
+			(effects
+				(font
+					(size 1.27 1.27)
+				)
+				(justify left)
+			)
+		)
+		(property "Footprint" ""
+			(at 38.1 47.244 0)
+			(effects
+				(font
+					(size 1.27 1.27)
+				)
+				(hide yes)
+			)
+		)
+		(property "Datasheet" "~"
+			(at 38.1 47.244 0)
+			(effects
+				(font
+					(size 1.27 1.27)
+				)
+				(hide yes)
+			)
+		)
+		(property "Description" ""
+			(at 38.1 47.244 0)
+			(effects
+				(font
+					(size 1.27 1.27)
+				)
+				(hide yes)
+			)
+		)
+		(pin "1"
+		)
+		(instances
+			(project "EVAL_TOLT_DC48V_3KW"
+				(path "/ab32ac57-1c18-4307-8f91-d2778314d165/2485f593-b019-439d-890e-42320f426831"
+					(reference "#FLG03")
+					(unit 1)
+				)
