File: EVAL-TOLT-DC48V-3KW-TOBO2-1206/DC-DC Buck Converter.kicad_sch (KiCad schematic)
At the start: 22 parts, among them IC1 LM5013QDDARQ1, J5 +5V_EXT

Commit message: v06112024
Parts:
- added J3: EXT/ITN 12V, Misc-Footprints:J3, symbol TSW-103-08-L-S:TSW-103-08-L-S
- added J4: +12V_EXT, Misc-Footprints:J4, symbol 1725656:1725656
- C13: footprint Kap-1206-Footprints:C13 -> Capacitor_SMD:C_1206_3216Metric
- C14, C16: footprint Kap-1206-Footprints:C14 -> Capacitor_SMD:C_1206_3216Metric
- C15, C17: footprint Kap-1206-Footprints:C15 -> Capacitor_SMD:C_1206_3216Metric
- C506, C507: footprint Kap-1206-Footprints:C506 -> Capacitor_SMD:C_1206_3216Metric
- C508: footprint Kap-1206-Footprints:C508 -> Capacitor_SMD:C_1206_3216Metric
- R1: footprint Resistor-1206-Footprints:R1 -> Resistor_SMD:R_1206_3216Metric_Pad1.30x1.75mm_HandSolder
- R4: footprint Resistor-1206-Footprints:R4 -> Resistor_SMD:R_1206_3216Metric_Pad1.30x1.75mm_HandSolder
- R501: footprint Resistor-1206-Footprints:R501 -> Resistor_SMD:R_1206_3216Metric_Pad1.30x1.75mm_HandSolder
- R502: footprint Resistor-1206-Footprints:R502 -> Resistor_SMD:R_1206_3216Metric_Pad1.30x1.75mm_HandSolder
- R503: footprint Resistor-1206-Footprints:R503 -> Resistor_SMD:R_1206_3216Metric_Pad1.30x1.75mm_HandSolder
- R8: footprint Resistor-1206-Footprints:R8 -> Resistor_SMD:R_1206_3216Metric_Pad1.30x1.75mm_HandSolder
Connections:
- net 12V: now also J3.02; no longer C508.2 (C2), L1.2, R502.1
- net GNDREF: now also J4.1
- new net: C508.2 (C2), J3.01, L1.2, R502.1
- new net: J3.03, J4.2

Commit message: v10112024
Parts:
- added C505: 12061C225KAT2A, Capacitor_SMD:C_1206_3216Metric, symbol C506:12061C225KAT2A
- added C509: 12061C273KAT2A, Capacitor_SMD:C_1206_3216Metric, symbol C508:12061C273KAT2A
- added C510: 47 pF, 115 mOhm, Capacitor_SMD:C_1206_3216Metric_Pad1.33x1.80mm_HandSolder, symbol Device:C
- added C511: 3.3 nF, 332 mOhm, Capacitor_SMD:C_1206_3216Metric_Pad1.33x1.80mm_HandSolder, symbol Device:C
- added D1: 770 mV, 5.5 A, Diode_SMD:D_1206_3216Metric, symbol Device:D_Schottky_Filled
- added R504: 221 kOhm, Resistor_SMD:R_1206_3216Metric_Pad1.30x1.75mm_HandSolder, symbol Device:R
- J3: footprint Misc-Footprints:J3 -> Connector_PinHeader_2.54mm:PinHeader_1x03_P2.54mm_Vertical
- J4: footprint Misc-Footprints:J4 -> Connector_PinHeader_2.54mm:PinHeader_1x02_P2.54mm_Vertical
- L1: footprint Misc-Footprints:L1 -> Inductor_SMD:L_1206_3216Metric_Pad1.22x1.90mm_HandSolder
Connections:
- net GNDREF: now also C505.1, C509.1 (C1), D1.2 (A)
- net V_BAT+: now also C505.2
- net at C507.2, IC1.8 (SW), L1.1: now also D1.1 (K), R504.1
- net at IC1.5 (FB), R502.2, R503.1: now also C510.2
- net at C508.2 (C2), J3.01, L1.2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: now also C509.2 (C2), C511.2
- net 5V renamed +5V
- new net: C510.1, C511.1, R504.2
Other:
- moved on the sheet: C507, C508, J3, J4, L1, LED1, R4, R502, R503, TP1

Commit message: v10112024-2
Parts:
- C510, C511: footprint Capacitor_SMD:C_1206_3216Metric_Pad1.33x1.80mm_HandSolder -> Capacitor_SMD:C_1206_3216Metric
- J3: symbol TSW-103-08-L-S:TSW-103-08-L-S -> PCM_SL_Pin_Headers:PINHD_1x3_Male
- J4: symbol 1725656:1725656 -> PCM_SL_Pin_Headers:PINHD_1x2_Male
Connections:
- net 12V: now also J3.2; no longer J3.02
- net at C508.2 (C2), C509.2 (C2), C511.2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: now also J3.1; no longer J3.01
- net at J4.2: now also J3.3; no longer J3.03
Changed lines of the file:
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@@
 	(paper "A4")
 	(junction
-		(at 254 67.31)
-		(diameter 0)
-		(color 0 0 0 0)
-	)
-	(junction
 		(at 31.75 128.27)
 		(diameter 0)
@@
 	)
 	(junction
-		(at 242.57 55.88)
-		(diameter 0)
-		(color 0 0 0 0)
-	)
-	(junction
 		(at 69.85 39.37)
 		(diameter 0)
@@
 	)
 	(junction
+		(at 254 67.31)
+		(diameter 0)
+		(color 0 0 0 0)
+	)
+	(junction
 		(at 153.67 55.88)
 		(diameter 0)
@@
 		(color 0 0 0 0)
 	)
+	(junction
+		(at 242.57 55.88)
+		(diameter 0)
+		(color 0 0 0 0)
+	)
 	(no_connect
 		(at 130.81 60.96)
@@
 	(wire
 		(pts
-			(xy 254 53.34) (xy 254 67.31)
+			(xy 251.46 55.88) (xy 242.57 55.88)
 		)
 		(stroke
@@
 	(wire
 		(pts
-			(xy 251.46 55.88) (xy 251.46 53.34)
-		)
-		(stroke
-			(width 0)
-			(type default)
-		)
-	)
-	(wire
-		(pts
 			(xy 53.34 132.08) (xy 53.34 128.27)
 		)
@@
 	(wire
 		(pts
-			(xy 256.54 53.34) (xy 265.43 53.34)
+			(xy 254 53.34) (xy 254 67.31)
 		)
 		(stroke
@@
 	(wire
 		(pts
-			(xy 254 67.31) (xy 254 72.39)
+			(xy 214.63 81.28) (xy 214.63 85.09)
 		)
 		(stroke
@@
 	(wire
 		(pts
-			(xy 214.63 81.28) (xy 214.63 85.09)
+			(xy 267.97 53.34) (xy 280.67 53.34)
 		)
 		(stroke
@@
 	(wire
 		(pts
+			(xy 254 67.31) (xy 254 72.39)
+		)
+		(stroke
+			(width 0)
+			(type default)
+		)
+	)
+	(wire
+		(pts
 			(xy 69.85 36.83) (xy 69.85 39.37)
 		)
@@
 	(wire
 		(pts
-			(xy 69.85 50.8) (xy 69.85 48.26)
+			(xy 256.54 53.34) (xy 265.43 53.34)
 		)
 		(stroke
@@
 	(wire
 		(pts
-			(xy 132.08 81.28) (xy 189.23 81.28)
+			(xy 69.85 50.8) (xy 69.85 48.26)
 		)
 		(stroke
@@
 	(wire
 		(pts
-			(xy 31.75 148.59) (xy 31.75 157.48)
+			(xy 132.08 81.28) (xy 189.23 81.28)
 		)
 		(stroke
@@
 	(wire
 		(pts
-			(xy 99.06 139.7) (xy 99.06 151.13)
+			(xy 31.75 148.59) (xy 31.75 157.48)
 		)
 		(stroke
@@
 	(wire
 		(pts
-			(xy 195.58 128.27) (xy 209.55 128.27)
+			(xy 99.06 139.7) (xy 99.06 151.13)
 		)
 		(stroke
@@
 	(wire
 		(pts
-			(xy 267.97 53.34) (xy 280.67 53.34)
+			(xy 195.58 128.27) (xy 209.55 128.27)
 		)
 		(stroke
@@
 	(wire
 		(pts
-			(xy 242.57 55.88) (xy 251.46 55.88)
+			(xy 118.11 128.27) (xy 133.35 128.27)
 		)
 		(stroke
@@
 	(wire
 		(pts
-			(xy 118.11 128.27) (xy 133.35 128.27)
+			(xy 149.86 55.88) (xy 153.67 55.88)
 		)
 		(stroke
@@
 	(wire
 		(pts
-			(xy 149.86 55.88) (xy 153.67 55.88)
+			(xy 251.46 53.34) (xy 251.46 55.88)
 		)
 		(stroke
@@
 			)
 		)
-		(property "Footprint" "Capacitor_SMD:C_1206_3216Metric_Pad1.33x1.80mm_HandSolder"
+		(property "Footprint" "Capacitor_SMD:C_1206_3216Metric"
 			(at 201.93 68.8848 0)
 			(effects
@@
 	)
 	(symbol
-		(lib_id "TSW-103-08-L-S:TSW-103-08-L-S")
-		(at 254 40.64 90)
+		(lib_id "PCM_SL_Pin_Headers:PINHD_1x3_Male")
+		(at 254 49.53 90)
 		(unit 1)
 		(exclude_from_sim no)
@@
 		(dnp no)
 		(property "Reference" "J3"
-			(at 248.92 41.275 90)
+			(at 247.142 49.53 90)
 			(effects
 				(font
@@
 		)
 		(property "Value" "EXT/ITN 12V"
-			(at 248.92 43.18 90)
+			(at 247.904 46.228 90)
 			(effects
 				(font
@@
 		)
 		(property "Footprint" "Connector_PinHeader_2.54mm:PinHeader_1x03_P2.54mm_Vertical"
-			(at 254 40.64 0)
+			(at 259.08 48.26 0)
 			(effects
 				(font
 					(size 1.27 1.27)
 				)
-				(justify bottom)
 				(hide yes)
 			)
 		)
 		(property "Datasheet" ""
-			(at 254 40.64 0)
+			(at 245.11 49.53 0)
 			(effects
 				(font
@@
 			)
 		)
-		(property "Description" ""
-			(at 254 40.64 0)
+		(property "Description" "Pin Header male with pin space 2.54mm. Pin Count -3"
+			(at 254 49.53 0)
 			(effects
 				(font
@@
 		)
 		(property "PARTREV" "R"
-			(at 254 40.64 0)
+			(at 254 49.53 0)
 			(effects
 				(font
@@
 		)
 		(property "STANDARD" "Manufacturer Recommendations"
-			(at 254 40.64 0)
+			(at 254 49.53 0)
 			(effects
 				(font
@@
 		)
 		(property "MANUFACTURER" "Samtec"
-			(at 254 40.64 0)
+			(at 254 49.53 0)
 			(effects
 				(font
@@
 			)
 		)
-		(pin "01"
+		(pin "2"
 		)
-		(pin "02"
+		(pin "3"
 		)
-		(pin "03"
+		(pin "1"
 		)
 		(instances
@@
 	)
 	(symbol
-		(lib_name "1725656_1")
-		(lib_id "1725656:1725656")
-		(at 267.97 53.34 270)
+		(lib_id "PCM_SL_Pin_Headers:PINHD_1x2_Male")
+		(at 266.7 57.15 270)
 		(unit 1)
 		(exclude_from_sim no)
@@
 		(dnp no)
 		(property "Reference" "J4"
-			(at 269.24 57.15 90)
+			(at 271.018 57.15 90)
 			(effects
 				(font
@@
 		)
 		(property "Value" "+12V_EXT"
-			(at 267.335 62.23 90)
+			(at 266.7 60.452 90)
 			(effects
 				(font
@@
 		)
 		(property "Footprint" "Connector_PinHeader_2.54mm:PinHeader_1x02_P2.54mm_Vertical"
-			(at 362.89 36.83 0)
+			(at 262.89 58.42 0)
 			(effects
 				(font
 					(size 1.27 1.27)
 				)
-				(justify left top)
 				(hide yes)
 			)
 		)
 		(property "Datasheet" "https://www.phoenixcontact.com/online/portal/us/?uri=pxc-oc-itemdetail:pid=1725656&library=usen&pcck=P-11-01-05&tab=1&selectedCategory=ALL"
-			(at 462.89 36.83 0)
+			(at 274.32 57.15 0)
 			(effects
 				(font
 					(size 1.27 1.27)
 				)
-				(justify left top)
 				(hide yes)
 			)
 		)
-		(property "Description" ""
-			(at 267.97 53.34 0)
+		(property "Description" "Pin Header male with pin space 2.54mm. Pin Count -2"
+			(at 266.7 57.15 0)
 			(effects
 				(font
@@
 		)
 		(property "Height" "8.65"
-			(at 662.89 36.83 0)
+			(at 661.62 40.64 0)
 			(effects
 				(font
@@
 		)
 		(property "Manufacturer_Name" "Phoenix Contact"
-			(at 762.89 36.83 0)
+			(at 761.62 40.64 0)
 			(effects
 				(font
@@
 		)
 		(property "Manufacturer_Part_Number" "1725656"
-			(at 862.89 36.83 0)
+			(at 861.62 40.64 0)
 			(effects
 				(font
@@
 		)
 		(property "Mouser Part Number" "651-1725656"
-			(at 962.89 36.83 0)
+			(at 961.62 40.64 0)
 			(effects
 				(font
@@
 		)
 		(property "Mouser Price/Stock" "https://www.mouser.co.uk/ProductDetail/Phoenix-Contact/1725656?qs=Ul7CXFMnlWWQeccayYbRmw%3D%3D"
-			(at 1062.89 36.83 0)
+			(at 1061.62 40.64 0)
 			(effects
 				(font
@@
 		)
 		(property "Arrow Part Number" "1725656"
-			(at 1162.89 36.83 0)
+			(at 1161.62 40.64 0)
 			(effects
 				(font
@@
 		)
 		(property "Arrow Price/Stock" "https://www.arrow.com/en/products/1725656/phoenix-contact?region=nac"
-			(at 1262.89 36.83 0)
+			(at 1261.62 40.64 0)
 			(effects
 				(font
@@
 			)
 		)
-		(property "Footprint" "Capacitor_SMD:C_1206_3216Metric_Pad1.33x1.80mm_HandSolder"
+		(property "Footprint" "Capacitor_SMD:C_1206_3216Metric"
 			(at 190.1952 81.28 0)
 			(effects

Commit message: v11112024-3
Parts:
- TP1, TP2: footprint TestPoint:TestPoint_Bridge_Pitch2.54mm_Drill0.7mm -> TestPoint:TestPoint_Pad_3.0x3.0mm
Changed lines of the file:
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@@
 			)
 		)
-		(property "Footprint" "TestPoint:TestPoint_Bridge_Pitch2.54mm_Drill0.7mm"
+		(property "Footprint" "TestPoint:TestPoint_Pad_3.0x3.0mm"
 			(at 259.08 67.31 0)
 			(effects
@@
 			)
 		)
-		(property "Footprint" "TestPoint:TestPoint_Bridge_Pitch2.54mm_Drill0.7mm"
+		(property "Footprint" "TestPoint:TestPoint_Pad_3.0x3.0mm"
 			(at 200.66 124.46 0)
 			(effects

Commit message: v15112024
Parts:
- C506, C507: footprint Capacitor_SMD:C_1206_3216Metric -> Capacitor_SMD:C_1210_3225Metric_Pad1.33x2.70mm_HandSolder
- J4: footprint Connector_PinHeader_2.54mm:PinHeader_1x02_P2.54mm_Vertical -> Misc-Footprints:J4
Changed lines of the file:
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@@
 			)
 		)
-		(property "Footprint" "Capacitor_SMD:C_1206_3216Metric"
+		(property "Footprint" "Capacitor_SMD:C_1210_3225Metric_Pad1.33x2.70mm_HandSolder"
 			(at 140.97 64.77 0)
 			(effects
@@
 			)
 		)
-		(property "Footprint" "Capacitor_SMD:C_1206_3216Metric"
+		(property "Footprint" "Capacitor_SMD:C_1210_3225Metric_Pad1.33x2.70mm_HandSolder"
 			(at 69.85 45.72 0)
 			(effects
@@
 			)
 		)
-		(property "Footprint" "Connector_PinHeader_2.54mm:PinHeader_1x02_P2.54mm_Vertical"
+		(property "Footprint" "Misc-Footprints:J4"
 			(at 262.89 58.42 0)
 			(effects

Commit message: v15112024-3
Parts:
- removed D1: 770 mV, 5.5 A, Diode_SMD:D_1206_3216Metric, symbol Device:D_Schottky_Filled
- added D1: 770 mV, 5.5 A, Misc-Footprints:DPAK_SBRD10200_6P6X6P1_SDS, symbol SBRD10200:SBRD10200TR
- L1: footprint Inductor_SMD:L_1206_3216Metric_Pad1.22x1.90mm_HandSolder -> Misc-Footprints:L1
Connections:
- net GNDREF: now also D1.1 (ANODE), D1.3 (ANODE)
- net at C507.2, IC1.8 (SW), L1.1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: now also D1.2 (BASE_CATHODE)
Changed lines of the file:
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@@
 	)
 	(junction
-		(at 153.67 55.88)
-		(diameter 0)
-		(color 0 0 0 0)
-	)
-	(junction
 		(at 53.34 128.27)
 		(diameter 0)
@@
 	)
 	(junction
+		(at 162.306 55.88)
+		(diameter 0)
+		(color 0 0 0 0)
+	)
+	(junction
 		(at 95.25 128.27)
 		(diameter 0)
@@
 	)
 	(junction
+		(at 164.846 17.78)
+		(diameter 0)
+		(color 0 0 0 0)
+	)
+	(junction
 		(at 189.23 81.28)
 		(diameter 0)
@@
 	(wire
 		(pts
+			(xy 159.766 17.78) (xy 164.846 17.78)
+		)
+		(stroke
+			(width 0)
+			(type default)
+		)
+	)
+	(wire
+		(pts
 			(xy 254 104.14) (xy 254 111.76)
 		)
@@
 	(wire
 		(pts
-			(xy 153.67 55.88) (xy 173.99 55.88)
+			(xy 149.86 55.88) (xy 162.306 55.88)
 		)
 		(stroke
@@
 	(wire
 		(pts
+			(xy 162.306 53.34) (xy 162.306 55.88)
+		)
+		(stroke
+			(width 0)
+			(type default)
+		)
+	)
+	(wire
+		(pts
 			(xy 214.63 77.47) (xy 214.63 81.28)
 		)
@@
 	(wire
 		(pts
-			(xy 256.54 53.34) (xy 265.43 53.34)
+			(xy 162.306 55.88) (xy 173.99 55.88)
 		)
 		(stroke
@@
 	(wire
 		(pts
-			(xy 69.85 50.8) (xy 69.85 48.26)
+			(xy 256.54 53.34) (xy 265.43 53.34)
 		)
 		(stroke
@@
 	(wire
 		(pts
-			(xy 132.08 81.28) (xy 189.23 81.28)
+			(xy 69.85 50.8) (xy 69.85 48.26)
 		)
 		(stroke
@@
 	(wire
 		(pts
-			(xy 31.75 148.59) (xy 31.75 157.48)
+			(xy 132.08 81.28) (xy 189.23 81.28)
 		)
 		(stroke
@@
 	(wire
 		(pts
-			(xy 99.06 139.7) (xy 99.06 151.13)
+			(xy 31.75 148.59) (xy 31.75 157.48)
 		)
 		(stroke
@@
 	(wire
 		(pts
-			(xy 195.58 128.27) (xy 209.55 128.27)
+			(xy 99.06 139.7) (xy 99.06 151.13)
 		)
 		(stroke
@@
 	(wire
 		(pts
-			(xy 130.81 55.88) (xy 149.86 55.88)
+			(xy 195.58 128.27) (xy 209.55 128.27)
 		)
 		(stroke
@@
 	(wire
 		(pts
-			(xy 118.11 128.27) (xy 133.35 128.27)
+			(xy 130.81 55.88) (xy 149.86 55.88)
 		)
 		(stroke
@@
 	(wire
 		(pts
-			(xy 149.86 55.88) (xy 153.67 55.88)
+			(xy 118.11 128.27) (xy 133.35 128.27)
 		)
 		(stroke
@@
 	(wire
 		(pts
+			(xy 164.846 16.256) (xy 164.846 17.78)
+		)
+		(stroke
+			(width 0)
+			(type default)
+		)
+	)
+	(wire
+		(pts
 			(xy 69.85 39.37) (xy 69.85 40.64)
 		)
@@
 	)
 	(symbol
-		(lib_id "Device:D_Schottky_Filled")
-		(at 153.67 59.69 270)
-		(unit 1)
-		(exclude_from_sim no)
-		(in_bom yes)
-		(on_board yes)
-		(dnp no)
-		(fields_autoplaced yes)
-		(property "Reference" "D1"
-			(at 156.21 58.1024 90)
-			(effects
-				(font
-					(size 1.27 1.27)
-				)
-				(justify left)
-			)
-		)
-		(property "Value" "770 mV, 5.5 A"
-			(at 156.21 60.6424 90)
-			(effects
-				(font
-					(size 1.27 1.27)
-				)
-				(justify left)
-			)
-		)
-		(property "Footprint" "Diode_SMD:D_1206_3216Metric"
-			(at 153.67 59.69 0)
-			(effects
-				(font
-					(size 1.27 1.27)
-				)
-				(hide yes)
-			)
-		)
-		(property "Datasheet" "~"
-			(at 153.67 59.69 0)
-			(effects
-				(font
-					(size 1.27 1.27)
-				)
-				(hide yes)
-			)
-		)
-		(property "Description" "Schottky diode, filled shape"
-			(at 153.67 59.69 0)
-			(effects
-				(font
-					(size 1.27 1.27)
-				)
-				(hide yes)
-			)
-		)
-		(pin "2"
-		)
-		(pin "1"
-		)
-		(instances
-			(project "EVAL_TOLT_DC48V_3KW"
-				(path "/ab32ac57-1c18-4307-8f91-d2778314d165/9ee2cd02-96d7-461b-b7fb-170453b1d10b"
-					(reference "D1")
-					(unit 1)
-				)
-			)
-		)
-	)
-	(symbol
 		(lib_id "DC:LM5013QDDARQ1")
 		(at 95.25 55.88 0)
@@
 			)
 		)
-		(property "Footprint" "Inductor_SMD:L_1206_3216Metric_Pad1.22x1.90mm_HandSolder"
+		(property "Footprint" "Misc-Footprints:L1"
 			(at 189.23 55.88 0)
 			(effects
@@
 	)
 	(symbol
-		(lib_id "power:GNDREF")
-		(at 153.67 63.5 0)
+		(lib_id "SBRD10200:SBRD10200TR")
+		(at 164.846 17.78 270)
 		(unit 1)
 		(exclude_from_sim no)
@@
 		(dnp no)
 		(fields_autoplaced yes)
-		(property "Reference" "#PWR028"
-			(at 153.67 69.85 0)
+		(property "Reference" "D1"
+			(at 168.91 34.2899 90)
 			(effects
 				(font
 					(size 1.27 1.27)
 				)
-				(hide yes)
+				(justify left)
 			)
 		)
-		(property "Value" "GNDREF"
-			(at 153.67 68.58 0)
+		(property "Value" "770 mV, 5.5 A"
+			(at 168.91 36.8299 90)
 			(effects
 				(font
 					(size 1.27 1.27)
 				)
+				(justify left)
 			)
 		)
-		(property "Footprint" ""
-			(at 153.67 63.5 0)
+		(property "Footprint" "Misc-Footprints:DPAK_SBRD10200_6P6X6P1_SDS"
+			(at 178.689 17.907 0)
 			(effects
 				(font
 					(size 1.27 1.27)
+					(italic yes)
 				)
 				(hide yes)
 			)
 		)
-		(property "Datasheet" ""
-			(at 153.67 63.5 0)
+		(property "Datasheet" "SBRD10200TR"
+			(at 174.498 18.161 0)
 			(effects
 				(font
 					(size 1.27 1.27)
+					(italic yes)
 				)
 				(hide yes)
 			)
 		)
-		(property "Description" "Power symbol creates a global label with name \"GNDREF\" , reference supply ground"
-			(at 153.67 63.5 0)
+		(property "Description" "Schottky diode, filled shape"
+			(at 184.912 15.367 0)
 			(effects
 				(font
@@
 			)
 		)
+		(pin "2"
+		)
 		(pin "1"
 		)
+		(pin "3"
+		)
 		(instances
 			(project "EVAL_TOLT_DC48V_3KW"
 				(path "/ab32ac57-1c18-4307-8f91-d2778314d165/9ee2cd02-96d7-461b-b7fb-170453b1d10b"
-					(reference "#PWR028")
+					(reference "D1")
 					(unit 1)
 				)
@@
 					(unit 1)
 				)
+			)
+		)
+	)
+	(symbol
+		(lib_id "power:GNDREF")
+		(at 164.846 16.256 180)
+		(unit 1)
+		(exclude_from_sim no)
+		(in_bom yes)
+		(on_board yes)
+		(dnp no)
+		(property "Reference" "#PWR033"
+			(at 164.846 9.906 0)
+			(effects
+				(font
+					(size 1.27 1.27)
+				)
+				(hide yes)
+			)
+		)
+		(property "Value" "GNDREF"
+			(at 170.434 16.51 0)
+			(effects
+				(font
+					(size 1.27 1.27)
+				)
+			)
+		)
+		(property "Footprint" ""
+			(at 164.846 16.256 0)
+			(effects
+				(font
+					(size 1.27 1.27)
+				)
+				(hide yes)
+			)
+		)
+		(property "Datasheet" ""
+			(at 164.846 16.256 0)
+			(effects
+				(font
+					(size 1.27 1.27)
+				)
+				(hide yes)
+			)
+		)
+		(property "Description" "Power symbol creates a global label with name \"GNDREF\" , reference supply ground"
+			(at 164.846 16.256 0)
+			(effects
+				(font
+					(size 1.27 1.27)
+				)
+				(hide yes)
+			)
+		)
+		(pin "1"
+		)
+		(instances
+			(project "EVAL_TOLT_DC48V_3KW"
+				(path "/ab32ac57-1c18-4307-8f91-d2778314d165/9ee2cd02-96d7-461b-b7fb-170453b1d10b"
+					(reference "#PWR033")
+					(unit 1)
+				)
